Commit message: Correct routes errors and add first version of inspection revision

File: robots/rb1_base.urdf.xacro (robot description, xacro)
@@ -57,8 +57,8 @@
 	<xacro:gazebo_colors prefix="$(arg prefix)"/>
 	<!-- WHEELS -->
-	<xacro:rubber_wheel prefix="$(arg prefix)right" parent="$(arg prefix)base_link" reflect="false" hq="${hq}">
+	<xacro:rubber_wheel prefix="$(arg prefix)right" parent="$(arg prefix)base_link" hq="${hq}">
 		<origin xyz="${wheel_offset_x} -${wheel_offset_y} ${wheel_offset_z}" rpy="0 0 0"/>
 	</xacro:rubber_wheel>
-	<xacro:rubber_wheel prefix="$(arg prefix)left" parent="$(arg prefix)base_link" reflect="true" hq="${hq}">
+	<xacro:rubber_wheel prefix="$(arg prefix)left" parent="$(arg prefix)base_link" hq="${hq}">
 		<origin xyz="${wheel_offset_x} ${wheel_offset_y} ${wheel_offset_z}" rpy="0 0 0"/>
 	</xacro:rubber_wheel>

File: robots/rbkairos_ur10e_plus.urdf.xacro (robot description, xacro)
@@ -59,5 +59,5 @@
     <!-- Here we create the robot elements using the xacro:macros imported at the beggining of this file -->
     <!-- Summit XL base -->
-    <xacro:summit_xl_steel_base prefix="$(arg prefix)" publish_bf="true" hq="${hq}" laser_support="true" />
+    <xacro:rbkairos_base prefix="$(arg prefix)" publish_bf="true" hq="${hq}" laser_support="true" />
     <xacro:omni_wheel prefix="$(arg prefix)front_right" parent="$(arg prefix)base_link" reflect="false" hq="${hq}">
       <origin xyz="${wheel_offset_x} -${wheel_offset_y} ${wheel_offset_z}" rpy="0 0 0"/>

File: robots/rbsherkan_std.urdf.xacro (robot description, xacro)
@@ -48,5 +48,15 @@
     </xacro:macro>
   <!-- Gazebo ros control pluggins -->
-  <xacro:ros_control namespace="robot" config_controllers="''"/>
+  <!-- ros control plugin -->
+  <xacro:macro name="ros_control">
+    <gazebo>
+      <plugin name="ros_control" filename="libgazebo_ros_control.so">
+		    <robotParam>robot_description</robotParam>
+        <controlPeriod>0.001</controlPeriod>
+	      <robotSimType>gazebo_ros_control/DefaultRobotHWSim</robotSimType>
+		    <legacyModeNS>true</legacyModeNS>
+      </plugin>
+    </gazebo>
+	</xacro:macro>
   <xacro:rbsherkan prefix="$(arg prefix)" hq="${hq}" />
 </robot>

File: urdf/arms/kinova/kinova_base.urdf.xacro (robot description, xacro)
@@ -15,5 +15,5 @@
        	  <origin xyz="0 0 0" rpy="0 0 0" />
 		  <geometry>
-			<mesh filename="package://rb1_base_description/meshes/arms/kinova/rb1_kinova_base-v1.dae" />
+			<mesh filename="package://robot_description/meshes/arms/kinova/rb1_kinova_base-v1.dae" />
 		  </geometry>
       </visual>
@@ -21,5 +21,5 @@
 		<origin xyz="0 0 0" rpy="${M_PI/2} 0 0" />
         <geometry>
-          <mesh filename="package://rb1_base_description/meshes/arms/kinova/rb1_kinova_base-v1.dae" />
+          <mesh filename="package://robot_description/meshes/arms/kinova/rb1_kinova_base-v1.dae" />
         </geometry>
       </collision>

File: urdf/arms/ur/torso_ur3.urdf.xacro (robot description, xacro)
@@ -15,5 +15,5 @@
        	<origin xyz="0 0 0" rpy="0 0 0" />
         <geometry>
-          <mesh filename="package://rb1_base_description/meshes/arms/ur/rb1_torso_ur3.dae" />
+          <mesh filename="package://robot_description/meshes/arms/ur/rb1_torso_ur3.dae" />
         </geometry>
       </visual>
@@ -21,5 +21,5 @@
 		    <origin xyz="0 0 0" rpy="${M_PI/2} 0 0" />
         <geometry>
-          <mesh filename="package://rb1_base_description/meshes/arms/ur/rb1_torso_ur3.dae" />
+          <mesh filename="package://robot_description/meshes/arms/ur/rb1_torso_ur3.dae" />
         </geometry>
       </collision>

File: urdf/bases/legacy/old_rb1_base_versions/rb1_base.urdf.xacro (robot description, xacro)
@@ -32,10 +32,10 @@
        <xacro:if value="${hq}">
        <geometry>
-         <mesh filename="package://rb1_base_description/meshes/bases/legacy/rb1_base/rb1v2_base.dae"/>
+         <mesh filename="package://robot_description/meshes/bases/legacy/rb1_base/rb1v2_base.dae"/>
        </geometry>
        </xacro:if>
        <xacro:unless value="${hq}">
        <geometry>
-       <mesh filename="package://rb1_base_description/meshes/bases/legacy/rb1_base/rb1v2_base.stl"/>
+       <mesh filename="package://robot_description/meshes/bases/legacy/rb1_base/rb1v2_base.stl"/>
        </geometry>
        </xacro:unless>
@@ -47,5 +47,5 @@
        <origin xyz="0 0 0" rpy="0 0 0 " />
        <geometry>
-         <mesh filename="package://rb1_base_description/meshes/bases/legacy/rb1_base/rb1v2_base.dae"/>
+         <mesh filename="package://robot_description/meshes/bases/legacy/rb1_base/rb1v2_base.dae"/>
        </geometry>
     </collision>
@@ -67,10 +67,10 @@
        <xacro:if value="${hq}">
        <geometry>
-	     <mesh filename="package://rb1_base_description/meshes/bases/legacy/rb1_base/rb1v2_front_cover.dae"/>
+	     <mesh filename="package://robot_description/meshes/bases/legacy/rb1_base/rb1v2_front_cover.dae"/>
        </geometry>
        </xacro:if>
        <xacro:unless value="${hq}">
        <geometry>
-       <mesh filename="package://rb1_base_description/meshes/bases/legacy/rb1_base/rb1v2_front_cover.stl"/>
+       <mesh filename="package://robot_description/meshes/bases/legacy/rb1_base/rb1v2_front_cover.stl"/>
        </geometry>
        </xacro:unless>
@@ -82,5 +82,5 @@
        <origin xyz="0 0 0" rpy="0 0 0 " />
        <geometry>
-         <mesh filename="package://rb1_base_description/meshes/bases/legacy/rb1_base/rb1v2_front_cover.dae"/>
+         <mesh filename="package://robot_description/meshes/bases/legacy/rb1_base/rb1v2_front_cover.dae"/>
        </geometry>
     </collision>

File: urdf/bases/legacy/old_rb1_base_versions/rb1_base_platform_kinova.urdf.xacro (robot description, xacro)
@@ -6,12 +6,12 @@
 	<!-- First we import all posible elements defined in the urdf.xacro files. All these elements are defined as macro:xacros -->
 	<!-- Import RB1 base elements -->
-    <xacro:include filename="$(find rb1_base_description)/urdf/bases/rb1_base_v3.urdf.xacro" /> <!-- v3 name from engineering department -->
+    <xacro:include filename="$(find robot_description)/urdf/bases/rb1_base_v3.urdf.xacro" /> <!-- v3 name from engineering department -->
 	<!-- Import RB1 wheels -->
-	<xacro:include filename="$(find rb1_base_description)/urdf/wheels/rubber_wheel/rubber_wheel_150.urdf.xacro" />
-	<xacro:include filename="$(find rb1_base_description)/urdf/wheels/omni_wheel/omni_wheel.urdf.xacro" />
+	<xacro:include filename="$(find robot_description)/urdf/wheels/rubber_wheel/rubber_wheel_150.urdf.xacro" />
+	<xacro:include filename="$(find robot_description)/urdf/wheels/omni_wheel/omni_wheel.urdf.xacro" />
 	<!-- Import all available sensors -->
 	<xacro:include filename="$(find robotnik_sensors)/urdf/all_sensors.urdf.xacro" />
     <!-- Import Elevator -->
-	<xacro:include filename="$(find rb1_base_description)/urdf/structures/elevator/rb1_base_elevator.urdf.xacro"/>
+	<xacro:include filename="$(find robot_description)/urdf/structures/elevator/rb1_base_elevator.urdf.xacro"/>
 	<!-- rb1_base -->
 	<xacro:macro name="rb1_base" params="prefix">

File: urdf/bases/legacy/old_rb1_base_versions/rb1_base_v0.urdf.xacro (robot description, xacro)
@@ -32,10 +32,10 @@
        <xacro:if value="${hq}">
        <geometry>
-         <mesh filename="package://rb1_base_description/meshes/bases/legacy/rb1_base/rb1v0_base.dae"/>
+         <mesh filename="package://robot_description/meshes/bases/legacy/rb1_base/rb1v0_base.dae"/>
        </geometry>
        </xacro:if>
        <xacro:unless value="${hq}">
        <geometry>
-       <mesh filename="package://rb1_base_description/meshes/bases/legacy/rb1_base/rb1v0_base.stl"/>
+       <mesh filename="package://robot_description/meshes/bases/legacy/rb1_base/rb1v0_base.stl"/>
        </geometry>
        </xacro:unless>
@@ -47,5 +47,5 @@
        <origin xyz="0 0 0" rpy="0 0 0 " />
        <geometry>
-         <mesh filename="package://rb1_base_description/meshes/bases/legacy/rb1_base/rb1v0_base.dae"/>
+         <mesh filename="package://robot_description/meshes/bases/legacy/rb1_base/rb1v0_base.dae"/>
        </geometry>
     </collision>

File: urdf/bases/legacy/old_rb1_base_versions/rb1_base_v1.urdf.xacro (robot description, xacro)
@@ -32,10 +32,10 @@
        <xacro:if value="${hq}">
        <geometry>
-	     <mesh filename="package://rb1_base_description/meshes/bases/legacy/rb1_base/rb1v1_base.dae"/>
+	     <mesh filename="package://robot_description/meshes/bases/legacy/rb1_base/rb1v1_base.dae"/>
        </geometry>
        </xacro:if>
        <xacro:unless value="${hq}">
        <geometry>
-       <mesh filename="package://rb1_base_description/meshes/bases/legacy/rb1_base/rb1v1_base.stl"/>
+       <mesh filename="package://robot_description/meshes/bases/legacy/rb1_base/rb1v1_base.stl"/>
        </geometry>
        </xacro:unless>
@@ -47,5 +47,5 @@
        <origin xyz="0 0 0" rpy="0 0 0 " />
        <geometry>
-         <mesh filename="package://rb1_base_description/meshes/bases/legacy/rb1_base/rb1v1_base.dae"/>
+         <mesh filename="package://robot_description/meshes/bases/legacy/rb1_base/rb1v1_base.dae"/>
        </geometry>
     </collision>

File: urdf/bases/legacy/old_rb1_base_versions/rb1_base_v2.urdf.xacro (robot description, xacro)
@@ -32,10 +32,10 @@
        <xacro:if value="${hq}">
        <geometry>
-	     <mesh filename="package://rb1_base_description/meshes/bases/legacy/rb1_base/rb1v2_base.dae"/>
+	     <mesh filename="package://robot_description/meshes/bases/legacy/rb1_base/rb1v2_base.dae"/>
        </geometry>
        </xacro:if>
        <xacro:unless value="${hq}">
        <geometry>
-       <mesh filename="package://rb1_base_description/meshes/bases/legacy/rb1_base/rb1v2_base.stl"/>
+       <mesh filename="package://robot_description/meshes/bases/legacy/rb1_base/rb1v2_base.stl"/>
        </geometry>
        </xacro:unless>
@@ -47,5 +47,5 @@
        <origin xyz="0 0 0" rpy="0 0 0 " />
        <geometry>
-         <mesh filename="package://rb1_base_description/meshes/bases/legacy/rb1_base/rb1v2_base.dae"/>
+         <mesh filename="package://robot_description/meshes/bases/legacy/rb1_base/rb1v2_base.dae"/>
        </geometry>
     </collision>
@@ -67,10 +67,10 @@
        <xacro:if value="${hq}">
        <geometry>
-	     <mesh filename="package://rb1_base_description/meshes/bases/legacy/rb1_base/rb1v2_front_cover.dae"/>
+	     <mesh filename="package://robot_description/meshes/bases/legacy/rb1_base/rb1v2_front_cover.dae"/>
        </geometry>
        </xacro:if>
        <xacro:unless value="${hq}">
        <geometry>
-       <mesh filename="package://rb1_base_description/meshes/bases/legacy/rb1_base/rb1v2_front_cover.stl"/>
+       <mesh filename="package://robot_description/meshes/bases/legacy/rb1_base/rb1v2_front_cover.stl"/>
        </geometry>
        </xacro:unless>
@@ -82,5 +82,5 @@
        <origin xyz="0 0 0" rpy="0 0 0 " />
        <geometry>
-         <mesh filename="package://rb1_base_description/meshes/bases/legacy/rb1_base/rb1v2_front_cover.dae"/>
+         <mesh filename="package://robot_description/meshes/bases/legacy/rb1_base/rb1v2_front_cover.dae"/>
        </geometry>
     </collision>

File: urdf/bases/rb1_base_v3.urdf.xacro (robot description, xacro)
@@ -32,10 +32,10 @@
        <xacro:if value="${hq}">
        <geometry>
-	     <mesh filename="package://rb1_base_description/meshes/bases/rb1_base_v3.stl"/>
+	     <mesh filename="package://robot_description/meshes/bases/rb1_base_v3.stl"/>
        </geometry>
        </xacro:if>
        <xacro:unless value="${hq}">
        <geometry>
-       <mesh filename="package://rb1_base_description/meshes/bases/rb1_base_v3.stl"/>
+       <mesh filename="package://robot_description/meshes/bases/rb1_base_v3.stl"/>
        </geometry>
        </xacro:unless>
@@ -47,5 +47,5 @@
        <origin xyz="0 0 0" rpy="0 0 0 " />
        <geometry>
-         <mesh filename="package://rb1_base_description/meshes/bases/rb1_base_v3.dae"/>
+         <mesh filename="package://robot_description/meshes/bases/rb1_base_v3.dae"/>
        </geometry>
     </collision-->
@@ -67,10 +67,10 @@
        <xacro:if value="${hq}">
        <geometry>
-	     <mesh filename="package://rb1_base_description/meshes/bases/rb1_front_cover_v3.stl"/>
+	     <mesh filename="package://robot_description/meshes/bases/rb1_front_cover_v3.stl"/>
        </geometry>
        </xacro:if>
        <xacro:unless value="${hq}">
        <geometry>
-       <mesh filename="package://rb1_base_description/meshes/bases/rb1_front_cover_v3.stl"/>
+       <mesh filename="package://robot_description/meshes/bases/rb1_front_cover_v3.stl"/>
        </geometry>
        </xacro:unless>
@@ -82,5 +82,5 @@
        <origin xyz="0 0 0" rpy="0 0 0 " />
        <geometry>
-         <mesh filename="package://rb1_base_description/meshes/bases/rb1_front_cover_v3.dae"/>
+         <mesh filename="package://robot_description/meshes/bases/rb1_front_cover_v3.dae"/>
        </geometry>
     </collision>
@@ -102,10 +102,10 @@
        <xacro:if value="${hq}">
 		   <geometry>
-			 <mesh filename="package://rb1_base_description/meshes/bases/rb1_top_cover_v3.stl"/>
+			 <mesh filename="package://robot_description/meshes/bases/rb1_top_cover_v3.stl"/>
 		   </geometry>
        </xacro:if>
        <xacro:unless value="${hq}">
 		   <geometry>
-		   <mesh filename="package://rb1_base_description/meshes/bases/rb1_top_cover_v3.stl"/>
+		   <mesh filename="package://robot_description/meshes/bases/rb1_top_cover_v3.stl"/>
 		   </geometry>
        </xacro:unless>
@@ -117,5 +117,5 @@
        <origin xyz="0 0 0" rpy="0 0 0 " />
        <geometry>
-         <mesh filename="package://rb1_base_description/meshes/bases/rb1_top_cover_v3.dae"/>
+         <mesh filename="package://robot_description/meshes/bases/rb1_top_cover_v3.dae"/>
        </geometry>
     </collision>

File: urdf/wheels/omni_wheel/rb1_base_omni_wheel.urdf.xacro (robot description, xacro)
@@ -29,5 +29,5 @@
           <origin xyz="0 0 0" rpy="0 0 0" />
           <geometry>
-				<mesh filename="package://rb1_base_description/meshes/wheels/omni_wheel/legacy/rb1_base/rb1v2_omniwheel.dae" />
+				<mesh filename="package://robot_description/meshes/wheels/omni_wheel/rb1v2_omniwheel.dae" />
           </geometry>
         </xacro:if>

File: urdf/wheels/rubber_wheel/legacy/rb1_base_rubber_wheel.urdf.xacro (robot description, xacro)
@@ -30,8 +30,8 @@
 			<geometry>
 				<xacro:if value="${reflect}">
-					<mesh filename="package://robot_description/meshes/wheels/rubber_wheels/wheel_rubber_6inch.dae" />
+					<mesh filename="package://robot_description/meshes/wheels/rubber_wheel/wheel_rubber_6inch.dae" />
 				</xacro:if>
 				<xacro:unless value="${reflect}">
-					<mesh filename="package://robot_description/meshes/wheels/rubber_wheels/wheel_rubber_6inch.dae" />
+					<mesh filename="package://robot_description/meshes/wheels/rubber_wheel/wheel_rubber_6inch.dae" />
 				</xacro:unless>
 			</geometry>

File: urdf/wheels/rubber_wheel/legacy/rubber_wheel_140.urdf.xacro (robot description, xacro)
@@ -35,5 +35,5 @@
 				<geometry>
 					<!-- <cylinder length="${wheel_height}" radius="${wheel_radius}" /> -->
-					<mesh filename="package://robot_description/meshes/wheels/rubber_wheels/rubber_wheel_zltech.stl" />
+					<mesh filename="package://robot_description/meshes/wheels/rubber_wheel/rubber_wheel_zltech.stl" />
 				</geometry>
 			</visual>
@@ -46,5 +46,5 @@
 				</xacro:if>
 				<geometry>
-					<mesh filename="package://robot_description/meshes/wheels/rubber_wheels/rubber_wheel_zltech.stl" />
+					<mesh filename="package://robot_description/meshes/wheels/rubber_wheel/rubber_wheel_zltech.stl" />
 				</geometry>
 			</collision>

File: urdf/wheels/rubber_wheel/rbvogui_rubber_wheel.urdf.xacro (robot description, xacro)
@@ -52,8 +52,8 @@
           <geometry>
             <xacro:if value="${reflect}">
-              <mesh filename="package://robot_description/meshes/wheels/rubber_wheels/wheel_sxl.stl" />
+              <mesh filename="package://robot_description/meshes/wheels/rubber_wheel/wheel_sxl.stl" />
             </xacro:if>
             <xacro:unless value="${reflect}">
-              <mesh filename="package://robot_description/meshes/wheels/rubber_wheels/wheel_sxl.stl" />
+              <mesh filename="package://robot_description/meshes/wheels/rubber_wheel/wheel_sxl.stl" />
             </xacro:unless>
           </geometry>

File: urdf/wheels/rubber_wheel/rbvogui_xl_offroad_rubber_wheel_350mm.urdf.xacro (robot description, xacro)
@@ -56,5 +56,5 @@
           </xacro:unless>
           <geometry>
-            <mesh filename="package://robot_description/meshes/wheels/rubber_wheels/wheel_350mm.stl" />
+            <mesh filename="package://robot_description/meshes/wheels/rubber_wheel/wheel_350mm.stl" />
           </geometry>
         </xacro:if>

File: urdf/wheels/rubber_wheel/rbvogui_xl_rubber_wheel_285mm.urdf.xacro (robot description, xacro)
@@ -56,5 +56,5 @@
           </xacro:unless>
           <geometry>
-            <mesh filename="package://robot_description/meshes/wheels/rubber_wheels/wheel_285mm.stl" />
+            <mesh filename="package://robot_description/meshes/wheels/rubber_wheel/wheel_285mm.stl" />
           </geometry>
         </xacro:if>

File: urdf/wheels/rubber_wheel/rubber_wheel.urdf.xacro (robot description, xacro)
@@ -28,8 +28,8 @@
           <geometry>
 						<xacro:if value="${reflect}">
-							<mesh filename="package://robot_description/meshes/wheels/rubber_wheels/rubber_wheel_left.dae" />
+							<mesh filename="package://robot_description/meshes/wheels/rubber_wheel/rubber_wheel_left.dae" />
 						</xacro:if>
 						<xacro:unless value="${reflect}">
-							<mesh filename="package://robot_description/meshes/wheels/rubber_wheels/rubber_wheel_right.dae" />
+							<mesh filename="package://robot_description/meshes/wheels/rubber_wheel/rubber_wheel_right.dae" />
 						</xacro:unless>
           </geometry>
@@ -48,5 +48,5 @@
         <geometry>
           <!--cylinder length="${rubber_wheel_height}" radius="${rubber_wheel_radius}" /-->
-          <mesh filename="package://robot_description/meshes/wheels/rubber_wheels/rubber_wheel_right.dae" />
+          <mesh filename="package://robot_description/meshes/wheels/rubber_wheel/rubber_wheel_right.dae" />
         </geometry>
       </collision>
