Commit message: Update rubber_wheel mesh visualization format

File: robots/summit_xl_std.urdf.xacro (robot description, xacro)
@@ -29,4 +29,6 @@
 	<xacro:arg name="gps_longitude" default="0"/>
     <xacro:macro name="summit_xl" params="prefix publish_bf hq kinematics">
+	  <xacro:property name="mesh_file_left" value="robot_description/meshes/wheels/rubber_wheel/rubber_wheel_left" />
+	  <xacro:property name="mesh_file_right" value="robot_description/meshes/wheels/rubber_wheel/rubber_wheel_right" />
 		<!-- *************** -->
 		<!-- Robots Elements -->
@@ -36,14 +38,14 @@
 		<xacro:summit_xl_base prefix="$(arg prefix)" publish_bf="true" hq="${hq}" />
     <xacro:if value="${kinematics == 'skid' or kinematics == 'skid_4w'}">
-  		<xacro:rubber_wheel prefix="$(arg prefix)front_right" parent="$(arg prefix)base_link" reflect="false" hq="${hq}">
+  		<xacro:rubber_wheel prefix="$(arg prefix)front_right" parent="$(arg prefix)base_link" reflect="false" hq="${hq}" mesh_file="${mesh_file_right}">
   			<origin xyz="${wheel_offset_x} -${wheel_offset_y} ${wheel_offset_z}" rpy="0 0 0"/>
   		</xacro:rubber_wheel>
-  		<xacro:rubber_wheel prefix="$(arg prefix)front_left" parent="$(arg prefix)base_link" reflect="true" hq="${hq}">
+  		<xacro:rubber_wheel prefix="$(arg prefix)front_left" parent="$(arg prefix)base_link" reflect="false" hq="${hq}" mesh_file="${mesh_file_left}">
   			<origin xyz="${wheel_offset_x} ${wheel_offset_y} ${wheel_offset_z}" rpy="0 0 0"/>
   		</xacro:rubber_wheel>
-  		<xacro:rubber_wheel prefix="$(arg prefix)back_left" parent="$(arg prefix)base_link" reflect="true" hq="${hq}">
+  		<xacro:rubber_wheel prefix="$(arg prefix)back_left" parent="$(arg prefix)base_link" reflect="false" hq="${hq}" mesh_file="${mesh_file_left}">
   			<origin xyz="-${wheel_offset_x} ${wheel_offset_y} ${wheel_offset_z}" rpy="0 0 0"/>
   		</xacro:rubber_wheel>
-  		<xacro:rubber_wheel prefix="$(arg prefix)back_right" parent="$(arg prefix)base_link" reflect="false" hq="${hq}">
+  		<xacro:rubber_wheel prefix="$(arg prefix)back_right" parent="$(arg prefix)base_link" reflect="false" hq="${hq}" mesh_file="${mesh_file_right}">
   			<origin xyz="-${wheel_offset_x} -${wheel_offset_y} ${wheel_offset_z}" rpy="0 0 0"/>
   		</xacro:rubber_wheel>

File: urdf/bases/summit_hm_base.urdf.xacro (robot description, xacro)
@@ -13,9 +13,9 @@
 		<xacro:property name="docking_contact_offset_y" value="0.0" />
 		<xacro:property name="docking_contact_offset_z" value="0.03223" />
-		<xacro:property name="rubber_wheel_radius" value="0.13" />
+		<xacro:property name="rubber_wheel_radius" value="0.1397" />
 		<xacro:property name="rubber_wheel_width" value="0.12" />
-		<xacro:property name="rubber_wheel_mass" value="8" />
-		<xacro:property name="mesh_file_left" value="robot_description/meshes/wheels/rubber_wheel/rubber_wheel_v202311_left" />
-		<xacro:property name="mesh_file_right" value="robot_description/meshes/wheels/rubber_wheel/rubber_wheel_v202311_right" />
+		<xacro:property name="rubber_wheel_mass" value="11" />
+		<xacro:property name="mesh_file_left" value="robot_description/meshes/wheels/rubber_wheel/rubber_wheel_v5.3" />
+		<xacro:property name="mesh_file_right" value="robot_description/meshes/wheels/rubber_wheel/rubber_wheel_v5.3" />
 		<!-- BASE FOOTPRINT -->
 		<xacro:if value="${publish_bf}">
@@ -78,20 +78,20 @@
 		<xacro:rubber_wheel prefix="${prefix}front_right" parent="${prefix}base_link" reflect="false" hq="${hq}" rubber_wheel_radius="${rubber_wheel_radius}"
 							rubber_wheel_width="${rubber_wheel_width}" rubber_wheel_mass="${rubber_wheel_mass}"
-							mesh_file_left="${mesh_file_left}" mesh_file_right="${mesh_file_right}">
+							mesh_file="${mesh_file_right}">
 			<origin xyz="${wheel_offset_x} -${wheel_offset_y} ${wheel_offset_z}" rpy="0 0 0"/>
 		</xacro:rubber_wheel>
-		<xacro:rubber_wheel prefix="${prefix}front_left" parent="${prefix}base_link" reflect="true" hq="${hq}" rubber_wheel_radius="${rubber_wheel_radius}"
+		<xacro:rubber_wheel prefix="${prefix}front_left" parent="${prefix}base_link" reflect="false" hq="${hq}" rubber_wheel_radius="${rubber_wheel_radius}"
 							rubber_wheel_width="${rubber_wheel_width}" rubber_wheel_mass="${rubber_wheel_mass}"
-							mesh_file_left="${mesh_file_left}" mesh_file_right="${mesh_file_right}">
+							mesh_file="${mesh_file_left}">
 			<origin xyz="${wheel_offset_x} ${wheel_offset_y} ${wheel_offset_z}" rpy="0 0 0"/>
 		</xacro:rubber_wheel>
-		<xacro:rubber_wheel prefix="${prefix}back_left" parent="${prefix}base_link" reflect="true" hq="${hq}" rubber_wheel_radius="${rubber_wheel_radius}"
+		<xacro:rubber_wheel prefix="${prefix}back_left" parent="${prefix}base_link" reflect="false" hq="${hq}" rubber_wheel_radius="${rubber_wheel_radius}"
 							rubber_wheel_width="${rubber_wheel_width}" rubber_wheel_mass="${rubber_wheel_mass}"
-							mesh_file_left="${mesh_file_left}" mesh_file_right="${mesh_file_right}">
+							mesh_file="${mesh_file_left}">
 			<origin xyz="-${wheel_offset_x} ${wheel_offset_y} ${wheel_offset_z}" rpy="0 0 0"/>
 		</xacro:rubber_wheel>
 		<xacro:rubber_wheel prefix="${prefix}back_right" parent="${prefix}base_link" reflect="false" hq="${hq}" rubber_wheel_radius="${rubber_wheel_radius}"
 							rubber_wheel_width="${rubber_wheel_width}" rubber_wheel_mass="${rubber_wheel_mass}"
-							mesh_file_left="${mesh_file_left}" mesh_file_right="${mesh_file_right}">
+							mesh_file="${mesh_file_right}">
 			<origin xyz="-${wheel_offset_x} -${wheel_offset_y} ${wheel_offset_z}" rpy="0 0 0"/>
 		</xacro:rubber_wheel>

File: urdf/wheels/rubber_wheel/rubber_wheel.urdf.xacro (robot description, xacro)
@@ -8,6 +8,5 @@
   </xacro:macro>
   <xacro:macro name="rubber_wheel" params="prefix parent *origin reflect hq rubber_wheel_radius:=0.11 rubber_wheel_width:=0.15 rubber_wheel_mass:=6.5
-                                          mesh_file_left:=robot_description/meshes/wheels/rubber_wheel/rubber_wheel_left
-                                          mesh_file_right:=robot_description/meshes/wheels/rubber_wheel/rubber_wheel_right">
+                                          mesh_file:=robot_description/meshes/wheels/rubber_wheel/rubber_wheel_right">
 <!--WHEEL TIRE -->
     <joint name="${prefix}_wheel_joint" type="continuous">
@@ -23,12 +22,12 @@
         <!-- HIGH RESOLUTION WHEELS -->
         <xacro:if value="${hq}">
-          <origin xyz="0 0 0" rpy="0 0 0" />
+          <xacro:unless value="${reflect}">
+            <origin xyz="0 0 0" rpy="0 0 0" />
+          </xacro:unless>
+          <xacro:if value="${reflect}">
+            <origin xyz="0 0 0" rpy="${M_PI} 0 0" />
+          </xacro:if>
           <geometry>
-						<xacro:if value="${reflect}">
-							<mesh filename="package://${mesh_file_left}.dae" />
-						</xacro:if>
-						<xacro:unless value="${reflect}">
-							<mesh filename="package://${mesh_file_right}.dae" />
-						</xacro:unless>
+							<mesh filename="package://${mesh_file}.dae" />
           </geometry>
         </xacro:if>
@@ -42,12 +41,12 @@
       </visual>
       <collision>
-        <origin xyz="0 0 0" rpy="0 0 0" />
-        <geometry>
+          <xacro:unless value="${reflect}">
+            <origin xyz="0 0 0" rpy="0 0 0" />
+          </xacro:unless>
           <xacro:if value="${reflect}">
-							<mesh filename="package://${mesh_file_left}.stl" />
-						</xacro:if>
-						<xacro:unless value="${reflect}">
-							<mesh filename="package://${mesh_file_right}.stl" />
-          </xacro:unless>
+            <origin xyz="0 0 0" rpy="${M_PI} 0 0" />
+          </xacro:if>
+          <geometry>
+						<mesh filename="package://${mesh_file}.stl" />
         </geometry>
       </collision>
