Commit message: summit_hm_std.urdf.xacro: Add sensors position to xacro

File: robots/summit_hm_std.urdf.xacro (robot description, xacro)
@@ -24,7 +24,8 @@
 		<xacro:property name="top_structure_y" value="0"/>
 		<xacro:property name="top_structure_z" value="0.27998"/>
-		<xacro:property name="top_lidar_structure_x" value="-0.11924"/>
+		<xacro:property name="top_lidar_structure_x" value="0"/>
 		<xacro:property name="top_lidar_structure_y" value="0"/>
 		<xacro:property name="top_lidar_structure_z" value="0.27609"/>
+		<xacro:property name="PI" value="3.1415926535897931"/>
 		<!-- *************** -->
 		<!-- Robots Elements -->
@@ -39,4 +40,31 @@
 			<origin xyz="${top_lidar_structure_x} ${top_lidar_structure_y} ${top_lidar_structure_z}" rpy="0 0 0"/>
 		</xacro:summit_hm_structure>
+    	<!-- IMU -->
+    	<xacro:sensor_imu prefix="$(arg prefix)imu" parent="$(arg prefix)base_link" topic="imu/data">
+    	  <origin xyz="0.0 0.0 0.10398" rpy="0 0 0"/>
+    	</xacro:sensor_imu>
+    	<!-- PTZ camera -->
+    	<xacro:sensor_link_750_nh prefix="$(arg prefix)ptz_camera" parent="$(arg prefix)base_link">
+    	  <origin xyz="0.20878 0 0.28738" rpy="0 0 0"/>
+    	</xacro:sensor_link_750_nh>
+    	<!-- Sensia camera -->
+    	<xacro:sensor_blk_arc prefix="$(arg prefix)sensia_camera" parent="$(arg prefix)base_link">
+    	  <origin xyz="0.00001 0 0.54098" rpy="0 0 0"/>
+    	</xacro:sensor_blk_arc>
+    	<!-- RGBD -->
+    	<xacro:sensor_intel_d435 prefix="$(arg prefix)front_rgbd_camera" parent="$(arg prefix)base_link" prefix_topic="front_rgbd_camera">
+		<origin xyz="0.30995 0.0 0.16097" rpy="0 0 0"/>
+    	</xacro:sensor_intel_d435>
+		<xacro:sensor_intel_d435 prefix="$(arg prefix)rear_rgbd_camera" parent="$(arg prefix)base_link" prefix_topic="front_rgbd_camera">
+		<origin xyz="-0.308 0.0 0.18308" rpy="0 ${-PI} 0"/>
+    	</xacro:sensor_intel_d435>
+        <!-- GPS -->
+        <xacro:sensor_ublox prefix="${prefix}gps" parent="${prefix}base_link" use_mast="false">
+            <origin xyz="-0.26135 0.249 0.787" rpy="0 0 0"/>
+        </xacro:sensor_ublox>
+    	<!-- LIDAR -->
+    	<xacro:sensor_rs_helios_16p prefix="$(arg prefix)top_3d_laser" prefix_topic="top_3d_laser" parent="$(arg prefix)base_link" gpu="false">
+    	  <origin xyz="0.0 0.0 0.38998" rpy="0 0 0"/>
+    	</xacro:sensor_rs_helios_16p>
 		<!-- Gazebo ros control pluggins -->
 		<xacro:ros_control/>

Commit message: Add antena 5G Teltonika

File: robots/summit_hm_std.urdf.xacro (robot description, xacro)
@@ -8,4 +8,5 @@
 	<xacro:include filename="$(find robot_description)/urdf/bases/summit_hm_base.urdf.xacro" />
 	<xacro:include filename="$(find robot_description)/urdf/structures/summit_hm/summit_hm_structure.xacro" />
+	<xacro:include filename="$(find robot_description)/urdf/structures/sensor_support/antena-combo-5G-teltonika.urdf.xacro" />
 	<!-- Import all available sensors -->
 	<xacro:include filename="$(find robotnik_sensors)/urdf/all_sensors.urdf.xacro" />
@@ -61,5 +62,5 @@
         <!-- GPS -->
         <xacro:sensor_ublox prefix="${prefix}gps" parent="${prefix}base_link" use_mast="false">
-            <origin xyz="-0.26135 0.249 0.787" rpy="0 0 0"/>
+            <origin xyz="-0.26135 0.249 0.7671" rpy="0 0 0"/>
         </xacro:sensor_ublox>
     	<!-- LIDAR -->
@@ -67,4 +68,8 @@
     	  <origin xyz="0.0 0.0 0.38998" rpy="0 0 0"/>
     	</xacro:sensor_rs_helios_16p>
+		<!-- GPS -->
+		<xacro:sensor_antena_combo_5G_teltonika prefix="$(arg prefix)antenna" parent="$(arg prefix)base_link" gps_latitude="$(arg gps_latitude)" gps_longitude="$(arg gps_longitude)">
+			<origin xyz="-0.26135 -0.249 0.597" rpy="0 0 0"/>
+		</xacro:sensor_antena_combo_5G_teltonika>
 		<!-- Gazebo ros control pluggins -->
 		<xacro:ros_control/>

Commit message: Update summit_hm standard components

File: robots/summit_hm_std.urdf.xacro (robot description, xacro)
@@ -19,4 +19,5 @@
 	<xacro:arg name="gps_latitude" default="0"/>
 	<xacro:arg name="gps_longitude" default="0"/>
+	<xacro:arg name="sim_control_period" default="0.004"/>
     <xacro:macro name="summit_hm" params="prefix publish_bf hq kinematics:=skid">
 		<xacro:property name="top_structure_mesh" value="robot_description/meshes/structures/summit_hm/summit_hm_top_structure" />
@@ -27,5 +28,5 @@
 		<xacro:property name="top_lidar_structure_x" value="0"/>
 		<xacro:property name="top_lidar_structure_y" value="0"/>
-		<xacro:property name="top_lidar_structure_z" value="0.27609"/>
+		<xacro:property name="top_lidar_structure_z" value="0.38998"/>
 		<xacro:property name="PI" value="3.1415926535897931"/>
 		<!-- *************** -->
@@ -45,33 +46,25 @@
     	  <origin xyz="0.0 0.0 0.10398" rpy="0 0 0"/>
     	</xacro:sensor_imu>
-    	<!-- PTZ camera -->
-    	<xacro:sensor_link_750_nh prefix="$(arg prefix)ptz_camera" parent="$(arg prefix)base_link">
-    	  <origin xyz="0.20878 0 0.28738" rpy="0 0 0"/>
-    	</xacro:sensor_link_750_nh>
-    	<!-- Sensia camera -->
-    	<xacro:sensor_blk_arc prefix="$(arg prefix)sensia_camera" parent="$(arg prefix)base_link">
-    	  <origin xyz="0.00001 0 0.54098" rpy="0 0 0"/>
-    	</xacro:sensor_blk_arc>
     	<!-- RGBD -->
     	<xacro:sensor_intel_d435 prefix="$(arg prefix)front_rgbd_camera" parent="$(arg prefix)base_link" prefix_topic="front_rgbd_camera">
 		<origin xyz="0.30995 0.0 0.16097" rpy="0 0 0"/>
     	</xacro:sensor_intel_d435>
-		<xacro:sensor_intel_d435 prefix="$(arg prefix)rear_rgbd_camera" parent="$(arg prefix)base_link" prefix_topic="front_rgbd_camera">
+		<!--xacro:sensor_intel_d435 prefix="$(arg prefix)rear_rgbd_camera" parent="$(arg prefix)base_link" prefix_topic="rear_rgbd_camera">
 		<origin xyz="-0.308 0.0 0.18308" rpy="0 ${-PI} 0"/>
-    	</xacro:sensor_intel_d435>
+    	</xacro:sensor_intel_d435-->
         <!-- GPS -->
-        <xacro:sensor_ublox prefix="${prefix}gps" parent="${prefix}base_link" use_mast="false">
+        <xacro:sensor_ublox prefix="${prefix}gps" parent="${prefix}base_link" use_mast="false" include_inertial="false">
             <origin xyz="-0.26135 0.249 0.7671" rpy="0 0 0"/>
         </xacro:sensor_ublox>
     	<!-- LIDAR -->
-    	<xacro:sensor_rs_helios_16p prefix="$(arg prefix)top_3d_laser" prefix_topic="top_3d_laser" parent="$(arg prefix)base_link" gpu="false">
+    	<xacro:sensor_rs_helios_16p prefix="$(arg prefix)top_3d_laser" prefix_topic="top_3d_laser" parent="$(arg prefix)base_link" gpu="$(arg gpu)">
     	  <origin xyz="0.0 0.0 0.38998" rpy="0 0 0"/>
     	</xacro:sensor_rs_helios_16p>
-		<!-- GPS -->
+		<!-- Antenna -->
 		<xacro:sensor_antena_combo_5G_teltonika prefix="$(arg prefix)antenna" parent="$(arg prefix)base_link" gps_latitude="$(arg gps_latitude)" gps_longitude="$(arg gps_longitude)">
 			<origin xyz="-0.26135 -0.249 0.597" rpy="0 0 0"/>
 		</xacro:sensor_antena_combo_5G_teltonika>
 		<!-- Gazebo ros control pluggins -->
-		<xacro:ros_control/>
+		<xacro:ros_control control_period="$(arg sim_control_period)"/>
 		<xacro:if value="$(arg ros_planar_move_plugin)">
 			<xacro:skid_steering prefix="${prefix}" publish_tf="true" force_based="$(arg ros_planar_move_plugin_force_based)"/>

Commit message: fix summit hm xacro

File: robots/summit_hm_std.urdf.xacro (robot description, xacro)
@@ -12,5 +12,5 @@
 	<xacro:include filename="$(find robotnik_sensors)/urdf/all_sensors.urdf.xacro" />
 	<!-- Flag to select the high or low quality model -->
-	<xacro:arg name="prefix" default="robot_"/>
+	<xacro:arg name="prefix" default=""/>
 	<xacro:arg name="ros_planar_move_plugin" default="false"/>
     <xacro:arg name="ros_planar_move_plugin_force_based" default="false"/>
@@ -43,31 +43,31 @@
 		</xacro:summit_hm_structure>
     	<!-- IMU -->
-    	<xacro:sensor_imu prefix="$(arg prefix)imu" parent="$(arg prefix)base_link" topic="imu/data">
+    	<xacro:sensor_vectornav frame_prefix="$(arg prefix)imu_" parent="$(arg prefix)base_link" topic_prefix="imu/data">
     	  <origin xyz="0.0 0.0 0.10398" rpy="0 0 0"/>
-    	</xacro:sensor_imu>
+    	</xacro:sensor_vectornav>
     	<!-- RGBD -->
-    	<xacro:sensor_intel_d435 prefix="$(arg prefix)front_rgbd_camera" parent="$(arg prefix)base_link" prefix_topic="front_rgbd_camera">
+    	<xacro:sensor_intel_realsense_d435 frame_prefix="$(arg prefix)front_rgbd_camera_" parent="$(arg prefix)base_link" topic_prefix="front_rgbd_camera">
 		<origin xyz="0.30995 0.0 0.16097" rpy="0 0 0"/>
-    	</xacro:sensor_intel_d435>
-		<!--xacro:sensor_intel_d435 prefix="$(arg prefix)rear_rgbd_camera" parent="$(arg prefix)base_link" prefix_topic="rear_rgbd_camera">
+    	</xacro:sensor_intel_realsense_d435>
+		<xacro:sensor_intel_realsense_d435 frame_prefix="$(arg prefix)rear_rgbd_camera_" parent="$(arg prefix)base_link" topic_prefix="rear_rgbd_camera">
 		<origin xyz="-0.308 0.0 0.18308" rpy="0 ${-PI} 0"/>
-    	</xacro:sensor_intel_d435-->
+    	</xacro:sensor_intel_realsense_d435>
         <!-- GPS -->
-        <xacro:sensor_ublox prefix="${prefix}gps" parent="${prefix}base_link" use_mast="false">
+        <xacro:sensor_gps frame_prefix="${prefix}gps_" parent="${prefix}base_link">
             <origin xyz="-0.26135 0.249 0.7671" rpy="0 0 0"/>
-        </xacro:sensor_ublox>
+        </xacro:sensor_gps>
     	<!-- LIDAR -->
-    	<xacro:sensor_rs_helios_16p prefix="$(arg prefix)top_3d_laser" prefix_topic="top_3d_laser" parent="$(arg prefix)base_link" gpu="$(arg gpu)">
+    	<xacro:sensor_robosense_helios frame_prefix="$(arg prefix)top_3d_laser_" topic_prefix="top_3d_laser" parent="$(arg prefix)base_link" gpu="$(arg gpu)">
     	  <origin xyz="0.0 0.0 0.38998" rpy="0 0 0"/>
-    	</xacro:sensor_rs_helios_16p>
+    	</xacro:sensor_robosense_helios>
 		<!-- Antenna -->
-		<xacro:sensor_antena_combo_5G_teltonika prefix="$(arg prefix)antenna" parent="$(arg prefix)base_link" gps_latitude="$(arg gps_latitude)" gps_longitude="$(arg gps_longitude)">
+		<!-- <xacro:sensor_antena_combo_5G_teltonika prefix="$(arg prefix)antenna" parent="$(arg prefix)base_link" gps_latitude="$(arg gps_latitude)" gps_longitude="$(arg gps_longitude)">
 			<origin xyz="-0.26135 -0.249 0.597" rpy="0 0 0"/>
-		</xacro:sensor_antena_combo_5G_teltonika>
+		</xacro:sensor_antena_combo_5G_teltonika> -->
 		<!-- Gazebo ros control pluggins -->
-		<xacro:ros_control control_period="$(arg sim_control_period)"/>
-		<xacro:if value="$(arg ros_planar_move_plugin)">
-			<xacro:skid_steering prefix="${prefix}" publish_tf="true" force_based="$(arg ros_planar_move_plugin_force_based)"/>
-		</xacro:if>
+		<!-- <xacro:ros_control control_period="$(arg sim_control_period)"/> -->
+		<!-- <xacro:if value="$(arg ros_planar_move_plugin)"> -->
+			<!-- <xacro:skid_steering prefix="${prefix}" publish_tf="true" force_based="$(arg ros_planar_move_plugin_force_based)"/> -->
+		<!-- </xacro:if> -->
    </xacro:macro>
    <xacro:summit_hm prefix="$(arg prefix)" publish_bf="true" hq="true" kinematics="$(arg kinematics)"/>

File: urdf/bases/summit_hm_base.urdf.xacro (robot description, xacro)
@@ -80,4 +80,5 @@
 							mesh_file="${mesh_file_right}">
 			<origin xyz="${wheel_offset_x} -${wheel_offset_y} ${wheel_offset_z}" rpy="0 0 0"/>
+        	<axis xyz="0 -1 0" rpy="0 0 0" />
 		</xacro:rubber_wheel>
 		<xacro:rubber_wheel prefix="${prefix}front_left" parent="${prefix}base_link" reflect="false" hq="${hq}" rubber_wheel_radius="${rubber_wheel_radius}"
@@ -85,14 +86,17 @@
 							mesh_file="${mesh_file_left}">
 			<origin xyz="${wheel_offset_x} ${wheel_offset_y} ${wheel_offset_z}" rpy="0 0 0"/>
+        	<axis xyz="0 1 0" rpy="0 0 0" />
 		</xacro:rubber_wheel>
-		<xacro:rubber_wheel prefix="${prefix}back_left" parent="${prefix}base_link" reflect="false" hq="${hq}" rubber_wheel_radius="${rubber_wheel_radius}"
+		<xacro:rubber_wheel prefix="${prefix}rear_left" parent="${prefix}base_link" reflect="false" hq="${hq}" rubber_wheel_radius="${rubber_wheel_radius}"
 							rubber_wheel_width="${rubber_wheel_width}" rubber_wheel_mass="${rubber_wheel_mass}"
 							mesh_file="${mesh_file_left}">
 			<origin xyz="-${wheel_offset_x} ${wheel_offset_y} ${wheel_offset_z}" rpy="0 0 0"/>
+        	<axis xyz="0 1 0" rpy="0 0 0" />
 		</xacro:rubber_wheel>
-		<xacro:rubber_wheel prefix="${prefix}back_right" parent="${prefix}base_link" reflect="false" hq="${hq}" rubber_wheel_radius="${rubber_wheel_radius}"
+		<xacro:rubber_wheel prefix="${prefix}rear_right" parent="${prefix}base_link" reflect="false" hq="${hq}" rubber_wheel_radius="${rubber_wheel_radius}"
 							rubber_wheel_width="${rubber_wheel_width}" rubber_wheel_mass="${rubber_wheel_mass}"
 							mesh_file="${mesh_file_right}">
 			<origin xyz="-${wheel_offset_x} -${wheel_offset_y} ${wheel_offset_z}" rpy="0 0 0"/>
+        	<axis xyz="0 -1 0" rpy="0 0 0" />
 		</xacro:rubber_wheel>
 	</xacro:macro>

File: urdf/wheels/rubber_wheel/rubber_wheel.urdf.xacro (robot description, xacro)
@@ -7,5 +7,5 @@
               izz="${m*(3*r*r+h*h)/12}" />
   </xacro:macro>
-  <xacro:macro name="rubber_wheel" params="prefix parent *origin reflect hq rubber_wheel_radius:=0.11 rubber_wheel_width:=0.15 rubber_wheel_mass:=6.5
+  <xacro:macro name="rubber_wheel" params="prefix parent *origin *axis reflect hq rubber_wheel_radius:=0.11 rubber_wheel_width:=0.15 rubber_wheel_mass:=6.5
                                           mesh_file:=robot_description/meshes/wheels/rubber_wheel/rubber_wheel_right">
 <!--WHEEL TIRE -->
@@ -14,5 +14,5 @@
       <child link="${prefix}_wheel"/>
       <xacro:insert_block name="origin" />
-      <axis xyz="0 1 0" rpy="0 0 0" />
+      <xacro:insert_block name="axis" />
       <limit effort="100" velocity="100"/>
       <joint_properties damping="0.0" friction="0.0"/>
