Commit message: update vogui and vogui xl

File: robots/rbvogui_std.urdf.xacro (robot description, xacro)
@@ -24,5 +24,5 @@
     <xacro:property name="hq" value="true" />
     <xacro:property name="publish_bf" value="true" />
-    <xacro:arg name="prefix" default="robot_" />
+    <xacro:arg name="prefix" default="" />
     <xacro:arg name="gpu" default="true" />
     <xacro:arg name="kinematics" default="omni" />
@@ -71,19 +71,19 @@
         <!-- SENSORS see robotnik_sensors for the specific configuration -->
         <!-- IMU -->
-        <xacro:sensor_vectornav prefix="${prefix}imu" parent="${prefix}chassis_link">
+    	<xacro:sensor_vectornav frame_prefix="${prefix}imu_" parent="$(arg prefix)chassis_link" topic_prefix="imu/data">
             <origin xyz="0.3 -0.3 0.0725" rpy="0 0 0"/>
         </xacro:sensor_vectornav>
-        <!-- Front Camera -->
+        <!-- Front Camera
         <xacro:sensor_orbbec_astra prefix="${prefix}front_rgbd_camera" parent="${prefix}chassis_link">
             <origin xyz="0.46462 0.0 0.18258" rpy="0 0 0"/>
-        </xacro:sensor_orbbec_astra>
-        <!-- GPS -->
+        </xacro:sensor_orbbec_astra>-->
+        <!-- GPS
         <xacro:sensor_ublox prefix="${prefix}gps" parent="${prefix}chassis_link" use_mast="true">
             <origin xyz="-0.3875 0.34553 0.3965" rpy="0 0 0"/>
-        </xacro:sensor_ublox>
-        <!-- 2d laser -->
+        </xacro:sensor_ublox>-->
+        <!-- 2d laser
         <xacro:sensor_sick_tim551 prefix="${prefix}front_laser" parent="${prefix}chassis_link" gpu="${gpu}" min_angle="${-PI/2}" max_angle="${PI/2}" prefix_topic="front_laser">
-            <origin xyz="0.53 0.0 -0.0245" rpy="${PI} 0 0"/> <!-- Verificar X -->
-        </xacro:sensor_sick_tim551>
+            <origin xyz="0.53 0.0 -0.0245" rpy="${PI} 0 0"/>
+        </xacro:sensor_sick_tim551> -->
         <!-- 3D Laser
         <xacro:sensor_rslidar_16 prefix="${prefix}top_3d_laser" parent="${prefix}chassis_link" prefix_topic="top_3d_laser" gpu="${gpu}">

File: robots/rbvogui_xl_std.urdf.xacro (robot description, xacro)
@@ -12,6 +12,6 @@
     <!-- Import rbvogui fix wheels -->
     <xacro:include filename="$(find robot_description)/urdf/wheels/fixed_wheel/rbvogui_fixed_wheel_xl.urdf.xacro" />
-    <!-- Import arm structure -->
-    <xacro:include filename="$(find robot_description)/urdf/arms/ur/bi_arm_support.urdf.xacro" />
+    <!-- Import arm structure
+    <xacro:include filename="$(find robot_description)/urdf/arms/ur/bi_arm_support.urdf.xacro" /> -->
     <!-- Structures -->
     <xacro:include filename="$(find robot_description)/urdf/structures/rbvogui_chassis/top_cover.urdf.xacro" />
@@ -32,5 +32,5 @@
     <xacro:property name="hq" value="true" />
     <xacro:property name="publish_bf" value="true" />
-    <xacro:arg name="prefix" default="robot_" />
+    <xacro:arg name="prefix" default="" />
     <xacro:arg name="gpu" default="false" />
     <xacro:arg name="kinematics" default="omni" />
@@ -79,5 +79,5 @@
         <!-- SENSORS see robotnik_sensors for the specific configuration -->
         <!-- IMU -->
-        <xacro:sensor_vectornav prefix="${prefix}imu" parent="${prefix}chassis_link">
+    	<xacro:sensor_vectornav frame_prefix="${prefix}imu_" parent="$(arg prefix)chassis_link" topic_prefix="imu/data">
             <origin xyz="0.3 -0.3 0.0725" rpy="0 0 0"/>
         </xacro:sensor_vectornav>
@@ -86,8 +86,8 @@
             <origin xyz="-0.472 0.40028 0.44044" rpy="0 0 0"/>
         </xacro:sensor_gps_mast>
-        <!-- Orbbec camera -->
+        <!-- Orbbec camera
         <xacro:sensor_orbbec_astra prefix="${prefix}front_rgbd_camera" parent="${prefix}chassis_link">
             <origin xyz="0.637 0.0 -0.036" rpy="0 0 0"/>
-        </xacro:sensor_orbbec_astra>
+        </xacro:sensor_orbbec_astra>-->
         <!-- Zed camera
         <xacro:sensor_zed prefix="${prefix}zed" parent="${prefix}chassis_link" model="zed2">
@@ -95,5 +95,5 @@
         </xacro:sensor_zed>
         -->
-        <!-- Laser sick support -->
+        <!-- Laser sick support
         <xacro:sick_support prefix="${prefix}sick_front_support" parent="${prefix}chassis_link">
             <origin xyz="0.472 0.3795 0.09788" rpy="0 ${90*PI/180} ${90*PI/180}"/>
@@ -101,6 +101,6 @@
         <xacro:sick_support prefix="${prefix}sick_rear_support" parent="${prefix}chassis_link">
             <origin xyz="-0.472 -0.3795 0.09788" rpy="0 ${90*PI/180} -${90*PI/180}"/>
-        </xacro:sick_support>
-        <!-- Laser sick protector -->
+        </xacro:sick_support> -->
+        <!-- Laser sick protector
         <xacro:sick_protector prefix="${prefix}sick_front_protector" parent="${prefix}chassis_link">
             <origin xyz="0.64542 0.39594 0.11073" rpy="0 0 -${45*PI/180}"/>
@@ -108,6 +108,6 @@
         <xacro:sick_protector prefix="${prefix}sick_rear_protector" parent="${prefix}chassis_link">
             <origin xyz="-0.64542 -0.39594 0.11073" rpy="0 0 ${135*PI/180}"/>
-        </xacro:sick_protector>
-        <!-- 2d laser -->
+        </xacro:sick_protector>-->
+        <!-- 2d laser
         <xacro:sensor_sick_microscan3 prefix="${prefix}front_laser" parent="${prefix}chassis_link" prefix_topic="front_laser" gpu="${gpu}">
             <origin xyz="0.64555 0.39595 0.16608" rpy="${PI} 0 ${45*PI/180}"/>
@@ -115,5 +115,5 @@
         <xacro:sensor_sick_microscan3 prefix="${prefix}rear_laser" parent="${prefix}chassis_link" prefix_topic="rear_laser" gpu="${gpu}">
             <origin xyz="-0.64555 -0.39985 0.16608" rpy="${PI} 0 -${135*PI/180}"/>
-        </xacro:sensor_sick_microscan3>
+        </xacro:sensor_sick_microscan3>-->
     </xacro:macro>
     <!-- Gazebo ros control pluggins -->
