Commit message: fix rbkairos minor issues and test controller

File: robots/summit_xls_std.urdf.xacro (robot description, xacro)
@@ -52,5 +52,5 @@
 		<!-- Here we create the robot elements using the xacro:macros imported at the beggining of this file -->
 		<!-- Summit XL base -->
-		<xacro:summit_xl_steel_base prefix="$(arg prefix)" publish_bf="true" hq="${hq}" />
+		<xacro:summit_xl_steel_base prefix="$(arg prefix)_" publish_bf="true" hq="${hq}" />
 		<xacro:omni_wheel prefix="$(arg prefix)front_right" parent="$(arg prefix)base_link" reflect="false" hq="${hq}">
 			<origin xyz="${wheel_offset_x} -${wheel_offset_y} ${wheel_offset_z}" rpy="0 0 0"/>

File: robots/versions/rb_kairos/rbkairos_base.urdf.xacro (robot description, xacro)
@@ -5,5 +5,5 @@
   <!-- ***************** -->
   <!-- First we import all posible elements defined in the urdf.xacro files. All these elements are defined as macro:xacros -->
-  <xacro:arg name="prefix" default="robot"/>
+  <xacro:arg name="prefix" default="robot_"/>
   <xacro:arg name="ros_planar_move_plugin" default="true"/>
   <xacro:arg name="use_gpu_for_simulation" default="false"/>
@@ -11,7 +11,10 @@
   <xacro:include filename="$(find robot_description)/urdf/bases/rbkairos_base.urdf.xacro" />
   <xacro:rbkairos_base prefix="$(arg prefix)" publish_bf="true" hq="true" gpu="$(arg use_gpu_for_simulation)"/>
-  <xacro:ros_control/>
+  <xacro:include filename="$(find robot_gazebo)/config/ros2_control_gazebo_rbkairos.urdf.xacro" />
+  <xacro:ros2_control prefix="robot" robot_id="robot" controllers="">
+  </xacro:ros2_control>
+  <!-- <xacro:ros_control/>
   <xacro:if value="$(arg ros_planar_move_plugin)">
     <xacro:omni_steering prefix="$(arg prefix)" publish_tf="true"/>
-  </xacro:if>
+  </xacro:if> -->
 </robot>

File: urdf/bases/rbkairos_base.urdf.xacro (robot description, xacro)
@@ -64,9 +64,9 @@
   		</xacro:omni_wheel>
           <!-- IMU -->
-  		<xacro:sensor_imu_hector prefix="$(arg prefix)imu" parent="$(arg prefix)base_link">
+        <xacro:sensor_vectornav prefix="${prefix}" parent="${prefix}base_link" topic="/robot/imu/data">
   			<origin xyz="${imu_offset_x} ${imu_offset_y} ${imu_offset_z}" rpy="0 0 0"/>
-  		</xacro:sensor_imu_hector>
+        </xacro:sensor_vectornav>
   		<!-- SENSORS -->
-  		<xacro:sensor_sick_s300 prefix="$(arg prefix)front_laser" parent="$(arg prefix)base_link" prefix_topic="front_laser" gpu="${gpu}">
+  		<!-- <xacro:sensor_sick_s300 prefix="$(arg prefix)front_laser" parent="$(arg prefix)base_link" prefix_topic="front_laser" gpu="${gpu}">
   			<origin xyz="${front_laser_offset_x} ${front_laser_offset_y} ${front_laser_offset_z}" rpy="0 ${-PI} ${3/4*PI}" />
   		</xacro:sensor_sick_s300>
@@ -74,7 +74,7 @@
   			<origin xyz="${rear_laser_offset_x} ${rear_laser_offset_y} ${rear_laser_offset_z}" rpy="0 ${-PI} ${-1/4*PI}" />
   		</xacro:sensor_sick_s300>
-  		<xacro:sensor_orbbec_astra prefix="$(arg prefix)front_rgbd_camera" parent="$(arg prefix)base_link" prefix_topic="front_rgbd_camera">
+  		<xacro:sensor_orbbec_astra prefix="$(arg prefix)front_rgbd_camera" parent="$(arg prefix)base_link" ns="$(arg prefix)">
   			<origin xyz="${front_rgbd_camera_offset_x} ${front_rgbd_camera_offset_y} ${front_rgbd_camera_offset_z}" rpy="0 0 0"/>
-  		</xacro:sensor_orbbec_astra>
+  		</xacro:sensor_orbbec_astra> -->
      </xacro:macro>
 </robot>

File: urdf/bases/summit_xl_steel_base.urdf.xacro (robot description, xacro)
@@ -33,10 +33,10 @@
       <xacro:if value="${hq}">
       <geometry>
-      <mesh filename="package://robot_description/meshes/bases/legacy/xls/summit_xls_chassis.stl"/>
+        <mesh filename="package://robot_description/meshes/bases/legacy/xls/summit_xls_chassis.stl"/>
       </geometry>
       </xacro:if>
       <xacro:unless value="${hq}">
       <geometry>
-      <mesh filename="package://robot_description/meshes/bases/legacy/xls/summit_xls_chassis.dae"/>
+        <mesh filename="package://robot_description/meshes/bases/legacy/xls/summit_xls_chassis.dae"/>
       </geometry>
       </xacro:unless>
@@ -60,5 +60,5 @@
     <origin xyz="0 0 0" rpy="0 0 0" />
     <geometry>
-    <mesh filename="package://robot_description/meshes/bases/legacy/xls/summit_xls_chapas_inox_tapas.stl"/>
+      <mesh filename="package://robot_description/meshes/bases/legacy/xls/summit_xls_chapas_inox_tapas.stl"/>
     </geometry>
     <material name="darkgrey">
@@ -77,5 +77,5 @@
     <origin xyz="0 0 0" rpy="0 0 0" />
     <geometry>
-    <mesh filename="package://robot_description/meshes/bases/legacy/xls/robotnik_logo_chasis.stl"/>
+      <mesh filename="package://robot_description/meshes/bases/legacy/xls/robotnik_logo_chasis.stl"/>
     </geometry>
     <material name="darkgrey">
@@ -94,5 +94,5 @@
     <origin xyz="0 0 0" rpy="0 0 0" />
     <geometry>
-    <mesh filename="package://robot_description/meshes/bases/legacy/xls/robotnik_logo_chasis.stl"/>
+      <mesh filename="package://robot_description/meshes/bases/legacy/xls/robotnik_logo_chasis.stl"/>
     </geometry>
     <material name="darkgrey">
@@ -111,5 +111,5 @@
     <origin xyz="0 0 0" rpy="0 0 0" />
     <geometry>
-    <mesh filename="package://robot_description/meshes/bases/legacy/xls/robotnik_logo_chasis.stl"/>
+      <mesh filename="package://robot_description/meshes/bases/legacy/xls/robotnik_logo_chasis.stl"/>
     </geometry>
     <material name="darkgrey">
@@ -128,5 +128,5 @@
     <origin xyz="0 0 0" rpy="0 0 0" />
     <geometry>
-    <mesh filename="package://robot_description/meshes/bases/legacy/xls/robotnik_logo_chasis.stl"/>
+      <mesh filename="package://robot_description/meshes/bases/legacy/xls/robotnik_logo_chasis.stl"/>
     </geometry>
     <material name="darkgrey">

File: urdf/wheels/omni_wheel/omni_wheel.urdf.xacro (robot description, xacro)
@@ -18,5 +18,5 @@
       <axis xyz="0 1 0" rpy="0 0 0" />
       <limit effort="100" velocity="100"/>
-      <joint_properties damping="0.0" friction="0.0"/>
+      <joint_properties damping="1.0" friction="1.0"/>
     </joint>
     <link name="${prefix}_wheel_link">
@@ -26,10 +26,10 @@
           <xacro:if value="${reflect}">
             <geometry>
-              <mesh filename="package://robot_description/meshes/wheels/omni_wheel/omni_wheel_1.dae" />
+              <mesh filename="package://robot_description/meshes/wheels/omni_wheel/wheel_omni_4inch.dae" />
             </geometry>
           </xacro:if>
           <xacro:unless value="${reflect}">
             <geometry>
-              <mesh filename="package://robot_description/meshes/wheels/omni_wheel/omni_wheel_2.dae" />
+              <mesh filename="package://robot_description/meshes/wheels/omni_wheel/wheel_omni_4inch.dae" />
             </geometry>
 		  </xacro:unless>
@@ -68,5 +68,5 @@
     </link>
     <!-- Transmission is important to link the joints and the controller (see summit_xl_control/config/summit_xl_control.yaml)-->
-    <transmission name="${prefix}_wheel_joint_trans">
+    <!-- <transmission name="${prefix}_wheel_joint_trans">
       <type>transmission_interface/SimpleTransmission</type>
       <joint name="${prefix}_wheel_joint" >
@@ -76,12 +76,12 @@
          <mechanicalReduction>1</mechanicalReduction>
       </actuator>
-    </transmission>
+    </transmission> -->
     <gazebo reference="${prefix}_wheel_link">
-		<mu1 value="0.0"/>
-		<mu2 value="0.0"/>
-		<kp value="10000000.0" />
-		<kd value="1.0" />
-		<fdir1 value="1 0 0"/>
-        <turnGravityOff>false</turnGravityOff>
+      <mu1>0.90</mu1>
+      <mu2>0.85</mu2>
+      <kp>2.75e6</kp>
+      <kd>8.25e1</kd>
+      <fdir1>0 0 0</fdir1>
+      <maxContacts>4</maxContacts>
     </gazebo>
   </xacro:macro>
