Commit message: Add rb1, use has_elevator for rb_theron and rb1_base, create legacy folder and restructure files

File: robots/rb_theron.urdf.xacro (robot description, xacro)
@@ -7,5 +7,5 @@
 	<!-- First we import all posible elements defined in the urdf.xacro files. All these elements are defined as macro:xacros -->
 	<!-- Import differential base elements -->
-	<xacro:include filename="$(find robot_description)/robots/rb_theron_base.urdf.xacro" />
+	<xacro:include filename="$(find robot_description)/urdf/bases/rb_theron_base.urdf.xacro" />
 	<!-- Import wheels -->
 	<xacro:include filename="$(find robot_description)/urdf/wheels/rubber_wheel_150.urdf.xacro" />
@@ -14,4 +14,6 @@
 	<!-- Import Gazebo Stuff -->
 	<xacro:include filename="$(find robot_description)/urdf/common.gazebo.xacro" />
+	<!-- Import Elevator -->
+	<xacro:include filename="$(find robot_description)/urdf/elevator/elevator.urdf.xacro"/>
 	<!-- ***************** -->
 	<!-- Global parameters -->
@@ -24,7 +26,10 @@
 	<!-- Flag to select the high or low quality model -->
 	<xacro:property name="hq" value="true" />
-	<!-- *************** -->
-	<!-- Robots Elements -->
-	<!-- *************** -->
+	<!-- ******************* -->
+	<!-- ELEVATOR PARAMETERS -->
+	<!-- ******************* -->
+	<xacro:property name="elevator_x" value="0.0" />
+	<xacro:property name="elevator_y" value="0.0" />
+	<xacro:property name="elevator_z" value="0.2238" />
 	<xacro:arg name="prefix" default="robot_"/>
 	<xacro:arg name="ros_planar_move_plugin" default="false"/>
@@ -34,5 +39,10 @@
 	<xacro:arg name="gps_latitude" default="0"/>
 	<xacro:arg name="gps_longitude" default="0"/>
+	<xacro:arg name="has_elevator" default="false"/>
 	<xacro:arg name="use_sim" default="false"/>
+	<!-- *************** -->
+	<!-- Robots Elements -->
+	<!-- *************** -->
+	<xacro:arg name="prefix" default="robot_"/>
 	<!-- Here we create the robot elements using the xacro:macros imported at the beggining of this file -->
 	<!-- base with wheels -->
@@ -45,5 +55,11 @@
   	</xacro:if>
 	<xacro:gazebo_colors prefix="$(arg prefix)"/>
-<!-- SENSORS -->
+	<!-- ELEVATOR_PLATFORM -->
+	<xacro:if value="$(arg has_elevator)">
+		<xacro:elevator_platform prefix="$(arg prefix)elevator" parent="$(arg prefix)base_link" hq="${hq}">
+			<origin xyz="${elevator_x} -${elevator_y} ${elevator_z}" rpy="1.5708 0 1.5708"/>
+		</xacro:elevator_platform>
+	</xacro:if>
+  <!-- SENSORS -->
   <!-- TODO: Moved 0.01 in x, otherwise the camera is still inside the robot -->
 	<!--xacro:sensor_orbbec_astra prefix="$(arg prefix)front_rgbd_camera" parent="$(arg prefix)base_link" prefix_topic="front_rgbd_camera">

File: urdf/structures/bi_arm_support.urdf.xacro (robot description, xacro)
@@ -51,6 +51,6 @@
       </joint>
       <xacro:ur10e_robot prefix="${prefix}left_arm_"
-                kinematics_parameters_file="$(find rbvogui_control)/config/calibration/ur10_calibration.yaml"
-                joint_limits_parameters_file="$(find rbvogui_control)/config/calibration/ur10_joint_limits.yaml">
+                kinematics_parameters_file="$(find robot_description)/robot_control/config/calibration/ur10_calibration.yaml"
+                joint_limits_parameters_file="$(find robot_description)/robot_control/config/calibration/ur10_joint_limits.yaml">
       </xacro:ur10e_robot>
     </xacro:if>
@@ -72,6 +72,6 @@
       </joint>
       <xacro:ur10e_robot prefix="${prefix}right_arm_"
-                kinematics_parameters_file="$(find rbvogui_control)/config/calibration/ur10_calibration.yaml"
-                joint_limits_parameters_file="$(find rbvogui_control)/config/calibration/ur10_joint_limits.yaml">
+                kinematics_parameters_file="$(find robot_description)/robot_control/config/calibration/ur10_calibration.yaml"
+                joint_limits_parameters_file="$(find robot_description)/robot_control/config/calibration/ur10_joint_limits.yaml">
       </xacro:ur10e_robot>
     </xacro:if>

Commit message: Create macros to standardize urdf

File: robots/rb_theron.urdf.xacro (robot description, xacro)
@@ -6,8 +6,6 @@
 	<!-- ***************** -->
 	<!-- First we import all posible elements defined in the urdf.xacro files. All these elements are defined as macro:xacros -->
-	<!-- Import differential base elements -->
-	<xacro:include filename="$(find robot_description)/urdf/bases/rb_theron_base.urdf.xacro" />
-	<!-- Import wheels -->
-	<xacro:include filename="$(find robot_description)/urdf/wheels/rubber_wheel/rubber_wheel_150.urdf.xacro" />
+	<!-- Import rbtheron macro -->
+	<xacro:include filename="$(find robot_description)/robots/macros/rb_theron_macro.xacro"/>
 	<!-- Import all available sensors -->
 	<xacro:include filename="$(find robotnik_sensors)/urdf/all_sensors.urdf.xacro" />
@@ -19,21 +17,16 @@
 	<!-- Global parameters -->
 	<!-- ***************** -->
+	<!-- Second we define all the parameters and arguments to customize the robot characteristics -->
 	<xacro:property name="PI" value="3.1415926535897931"/>
-	<!-- Wheel parameters -->
-	<!--xacro:property name="wheel_offset_x" value="0" />
-	<xacro:property name="wheel_offset_y" value="0.2516" />
-	<xacro:property name="wheel_offset_z" value="0.0" /-->
 	<!-- Flag to select the high or low quality model -->
 	<xacro:property name="hq" value="true" />
-	<!-- ******************* -->
 	<!-- ELEVATOR PARAMETERS -->
-	<!-- ******************* -->
 	<xacro:property name="elevator_x" value="0.0" />
 	<xacro:property name="elevator_y" value="0.0" />
 	<xacro:property name="elevator_z" value="0.2238" />
-	<xacro:arg name="prefix" default=""/>
+	<xacro:arg name="robot_id" default="rbtheron"/>
 	<xacro:arg name="ros_planar_move_plugin" default="false"/>
     <xacro:arg name="ros_planar_move_plugin_force_based" default="false"/>
-	<xacro:arg name="kinematics" default="skid"/>
+	<xacro:arg name="kinematics" default="omni"/>
 	<xacro:arg name="gpu" default="false"/>
 	<xacro:arg name="gps_latitude" default="0"/>
@@ -41,50 +34,51 @@
 	<xacro:arg name="has_elevator" default="false"/>
 	<xacro:arg name="use_sim" default="false"/>
-	<!-- *************** -->
-	<!-- Robots Elements -->
-	<!-- *************** -->
-	<!-- Here we create the robot elements using the xacro:macros imported at the beggining of this file -->
-	<!-- base with wheels -->
-	<xacro:rb_theron_base prefix="$(arg prefix)" hq="${hq}" use_sim="$(arg use_sim)"/>
-	<!-- Gazebo ros control pluggins -->
-	<!--xacro:ros_control namespace="$(arg namespace)"/-->
-	<xacro:ros_control/>
-	<xacro:if value="$(arg ros_planar_move_plugin)">
-    	<xacro:omni_steering prefix="$(arg prefix)" publish_tf="true"/>
-  	</xacro:if>
-	<xacro:gazebo_colors prefix="$(arg prefix)"/>
+	<!-- Wheel parameters -->
+	<xacro:property name="wheel_offset_x" value="0" />
+	<xacro:property name="wheel_offset_y" value="0.2516" />
+	<xacro:property name="wheel_offset_z" value="0.0" />
+	<!-- castor -->
+	<xacro:property name="castor_offset_x" value="0.235" />
+	<xacro:property name="castor_offset_y" value="0.1825" />
+	<xacro:property name="castor_offset_z" value="0.0448" />
+	<!-- omni -->
+	<xacro:property name="omni_wheel_offset_x" value="0.2175" />    <!-- x,y,z in translation from base_link to the center of the wheel -->
+	<xacro:property name="omni_wheel_offset_y" value="0.204" />
+	<xacro:property name="omni_wheel_offset_z" value="0.0" />
+	<!-- Here we create the robot using the xacro:macro imported at the beggining of this file -->
+	<xacro:rb_theron robot_id="$(arg robot_id)" publish_bf="true" hq="true" kinematics="$(arg kinematics)"/>
 	<!-- ELEVATOR_PLATFORM -->
 	<xacro:if value="$(arg has_elevator)">
-		<xacro:elevator_platform prefix="$(arg prefix)elevator" parent="$(arg prefix)base_link" hq="${hq}">
+		<xacro:elevator_platform robot_id="$(arg robot_id)_elevator" parent="$(arg robot_id)_base_link" hq="${hq}">
 			<origin xyz="${elevator_x} -${elevator_y} ${elevator_z}" rpy="1.5708 0 1.5708"/>
 		</xacro:elevator_platform>
 	</xacro:if>
-  <!-- SENSORS -->
+	<!-- SENSORS -->
   <!-- TODO: Moved 0.01 in x, otherwise the camera is still inside the robot -->
-	<!--xacro:sensor_orbbec_astra prefix="$(arg prefix)front_rgbd_camera" parent="$(arg prefix)base_link" prefix_topic="front_rgbd_camera">
+	<!-- <xacro:sensor_orbbec_astra robot_id="$(arg prefix)front_rgbd_camera" parent="$(arg prefix)base_link" prefix_topic="front_rgbd_camera">
 		<origin xyz="0.3305 0.0 0.1748" rpy="0 0 0"/>
-	</xacro:sensor_orbbec_astra-->
-	<xacro:sensor_intel_realsense_d435 frame_prefix="$(arg prefix)front_rgbd_camera_" parent="$(arg prefix)base_link" topic_prefix="front_rgbd_camera">
+	</xacro:sensor_orbbec_astra> -->
+	<!-- <xacro:sensor_intel_realsense_d435 frame_robot_id="$(arg prefix)front_rgbd_camera_" parent="$(arg prefix)base_link" topic_robot_id="front_rgbd_camera">
 		<origin xyz="0.3045 0.0 0.1898" rpy="0 0 0"/>
-	</xacro:sensor_intel_realsense_d435>
-	<!--xacro:sensor_intel_d435 prefix="$(arg prefix)rear_rgbd_camera" parent="$(arg prefix)base_link" prefix_topic="rear_rgbd_camera">
+	</xacro:sensor_intel_realsense_d435> -->
+	<!-- xacro:sensor_intel_d435 robot_id="$(arg prefix)rear_rgbd_camera" parent="$(arg prefix)base_link" prefix_topic="rear_rgbd_camera">
 		<origin xyz="-0.3045 0.0 0.1158" rpy="0 0 3.1416"/>
 	</xacro:sensor_intel_d435>
-	<xacro:sensor_imu_hector prefix="$(arg prefix)imu" parent="$(arg prefix)base_link">
+	<xacro:sensor_imu_hector robot_id="$(arg prefix)imu" parent="$(arg prefix)base_link">
 		<origin xyz="-0.1975 0.0 0.1598" rpy="0 0 0"/>
-	</xacro:sensor_imu_hector-->
-	<xacro:sensor_sick_nanoscan3 frame_prefix="$(arg prefix)front_laser_" parent="$(arg prefix)base_link" topic_prefix="front_laser">
+	</xacro:sensor_imu_hector -->
+	<!-- <xacro:sensor_sick_nanoscan3 frame_robot_id="$(arg prefix)front_laser_" parent="$(arg prefix)base_link" topic_robot_id="front_laser">
 		<origin xyz="0.2675 -0.215 0.1613" rpy="0 -3.1416 2.3562"/>
 	</xacro:sensor_sick_nanoscan3>
-	<xacro:sensor_sick_nanoscan3 frame_prefix="$(arg prefix)rear_laser_" parent="$(arg prefix)base_link" topic_prefix="rear_laser">
+	<xacro:sensor_sick_nanoscan3 frame_robot_id="$(arg prefix)rear_laser_" parent="$(arg prefix)base_link" topic_robot_id="rear_laser">
 		<origin xyz="-0.2675 0.215 0.1613" rpy="0 -3.1416 -0.7854"/>
-	</xacro:sensor_sick_nanoscan3>
-	<!--xacro:sensor_sick_nanoscan3 prefix="$(arg prefix)front_laser" parent="$(arg prefix)base_link" prefix_topic="front_laser" min_angle="-2.0507619" max_angle="2.0507619">
+	</xacro:sensor_sick_nanoscan3> -->
+	<!--xacro:sensor_sick_nanoscan3 robot_id="$(arg prefix)front_laser" parent="$(arg prefix)base_link" prefix_topic="front_laser" min_angle="-2.0507619" max_angle="2.0507619">
 		<origin xyz="0.250 0.0 0.1643" rpy="0 3.1416 3.1416"/>
 	</xacro:sensor_sick_nanoscan3-->
-	<!--xacro:sensor_sick_tim571 prefix="$(arg prefix)front_laser" parent="$(arg prefix)base_link" prefix_topic="front_laser" min_angle="-2.0507619" max_angle="2.0507619">
+	<!--xacro:sensor_sick_tim571 robot_id="$(arg prefix)front_laser" parent="$(arg prefix)base_link" prefix_topic="front_laser" min_angle="-2.0507619" max_angle="2.0507619">
 		<origin xyz="0.2675 -0.215 0.1613" rpy="0 -3.1416 2.3562"/>
 	</xacro:sensor_sick_tim571-->
-	<!--xacro:sensor_sick_tim571 prefix="$(arg prefix)rear_laser" parent="$(arg prefix)base_link" prefix_topic="rear_laser" min_angle="-2.0507619" max_angle="2.0507619">
+	<!--xacro:sensor_sick_tim571 robot_id="$(arg prefix)rear_laser" parent="$(arg prefix)base_link" prefix_topic="rear_laser" min_angle="-2.0507619" max_angle="2.0507619">
 		<origin xyz="-0.2675 0.215 0.1613" rpy="0 -3.1416 -0.7854"/>
 	</xacro:sensor_sick_tim571-->

File: robots/summit_xl_std.urdf.xacro (robot description, xacro)
@@ -4,22 +4,19 @@
 	<!-- Imported elements -->
 	<!-- ***************** -->
-	<!-- First we import all posible elements defined in the urdf.xacro files. All these elements are defined as macro:xacros -->
-	<!-- Import summit XL base elements -->
-	<xacro:include filename="$(find robot_description)/urdf/bases/summit_xl_base.urdf.xacro" />
-	<!-- Import summit XL wheels -->
-	<xacro:include filename="$(find robot_description)/urdf/wheels/rubber_wheel/rubber_wheel.urdf.xacro" />
-  <xacro:include filename="$(find robot_description)/urdf/wheels/omni_wheel/omni_wheel.urdf.xacro" />
+	<!-- First we import the robot and all the sensors. All these elements are defined as macro:xacros -->
+	<!-- Import summit XL macro -->
+	<xacro:include filename="$(find robot_description)/robots/macros/summit_xl_macro.xacro"/>
 	<!-- Import all available sensors -->
 	<xacro:include filename="$(find robotnik_sensors)/urdf/all_sensors.urdf.xacro" />
 	<!-- Import antenna -->
 	<xacro:include filename="$(find robot_description)/urdf/structures/sensor_support/structure_teltonika.urdf.xacro" />
+	<!-- ***************** -->
+	<!-- Global parameters -->
+	<!-- ***************** -->
+	<!-- Second we define all the parameters and arguments to customize the robot characteristics -->
 	<xacro:property name="PI" value="3.1415926535897931"/>
-	<!-- Wheel parameters -->
-	<xacro:property name="wheel_offset_x" value="0.229" />    <!-- x,y,z in translation from base_link to the center of the wheel -->
-	<xacro:property name="wheel_offset_y" value="0.235" />
-	<xacro:property name="wheel_offset_z" value="0.0" />
 	<!-- Flag to select the high or low quality model -->
 	<xacro:property name="hq" value="true" />
-	<xacro:arg name="prefix" default="summit_xl_"/>
+	<xacro:arg name="robot_id" default="summit_xl"/>
 	<xacro:arg name="ros_planar_move_plugin" default="false"/>
     <xacro:arg name="ros_planar_move_plugin_force_based" default="false"/>
@@ -28,76 +25,34 @@
 	<xacro:arg name="gps_latitude" default="0"/>
 	<xacro:arg name="gps_longitude" default="0"/>
-    <xacro:macro name="summit_xl" params="prefix publish_bf hq kinematics">
-	  <xacro:property name="mesh_file_left" value="robot_description/meshes/wheels/rubber_wheel/rubber_wheel_left" />
-	  <xacro:property name="mesh_file_right" value="robot_description/meshes/wheels/rubber_wheel/rubber_wheel_right" />
-		<!-- *************** -->
-		<!-- Robots Elements -->
-		<!-- *************** -->
-		<!-- Here we create the robot elements using the xacro:macros imported at the beggining of this file -->
-		<!-- Summit XL base -->
-		<xacro:summit_xl_base prefix="$(arg prefix)" publish_bf="true" hq="${hq}" />
-    <xacro:if value="${kinematics == 'skid' or kinematics == 'skid_4w'}">
-  		<xacro:rubber_wheel prefix="$(arg prefix)front_right" parent="$(arg prefix)base_link" reflect="false" hq="${hq}" mesh_file="${mesh_file_right}">
-  			<origin xyz="${wheel_offset_x} -${wheel_offset_y} ${wheel_offset_z}" rpy="0 0 0"/>
-  		</xacro:rubber_wheel>
-  		<xacro:rubber_wheel prefix="$(arg prefix)front_left" parent="$(arg prefix)base_link" reflect="false" hq="${hq}" mesh_file="${mesh_file_left}">
-  			<origin xyz="${wheel_offset_x} ${wheel_offset_y} ${wheel_offset_z}" rpy="0 0 0"/>
-  		</xacro:rubber_wheel>
-  		<xacro:rubber_wheel prefix="$(arg prefix)back_left" parent="$(arg prefix)base_link" reflect="false" hq="${hq}" mesh_file="${mesh_file_left}">
-  			<origin xyz="-${wheel_offset_x} ${wheel_offset_y} ${wheel_offset_z}" rpy="0 0 0"/>
-  		</xacro:rubber_wheel>
-  		<xacro:rubber_wheel prefix="$(arg prefix)back_right" parent="$(arg prefix)base_link" reflect="false" hq="${hq}" mesh_file="${mesh_file_right}">
-  			<origin xyz="-${wheel_offset_x} -${wheel_offset_y} ${wheel_offset_z}" rpy="0 0 0"/>
-  		</xacro:rubber_wheel>
-    </xacro:if>
-    <xacro:if value="${kinematics == 'omni' or kinematics == 'omni_4w'}">
-  		<xacro:omni_wheel prefix="$(arg prefix)front_right" parent="$(arg prefix)base_link" reflect="false" hq="${hq}">
-  			<origin xyz="${wheel_offset_x} -${wheel_offset_y} ${wheel_offset_z}" rpy="0 0 0"/>
-  		</xacro:omni_wheel>
-  		<xacro:omni_wheel prefix="$(arg prefix)front_left" parent="$(arg prefix)base_link" reflect="true" hq="${hq}">
-  			<origin xyz="${wheel_offset_x} ${wheel_offset_y} ${wheel_offset_z}" rpy="0 0 0"/>
-  		</xacro:omni_wheel>
-  		<xacro:omni_wheel prefix="$(arg prefix)back_left" parent="$(arg prefix)base_link" reflect="true" hq="${hq}">
-  			<origin xyz="-${wheel_offset_x} ${wheel_offset_y} ${wheel_offset_z}" rpy="0 0 0"/>
-  		</xacro:omni_wheel>
-  		<xacro:omni_wheel prefix="$(arg prefix)back_right" parent="$(arg prefix)base_link" reflect="false" hq="${hq}">
-  			<origin xyz="-${wheel_offset_x} -${wheel_offset_y} ${wheel_offset_z}" rpy="0 0 0"/>
-  		</xacro:omni_wheel>
-    </xacro:if>
-        <!-- IMU -->
-		<xacro:sensor_imu prefix="$(arg prefix)imu" parent="$(arg prefix)base_link" topic="imu/data_raw">
-			<origin xyz="0.0385 0.132 0.158" rpy="0 0 0"/>
-		</xacro:sensor_imu>
-		<!-- 3d laser -->
-		<xacro:sensor_rs_helios_16p prefix="$(arg prefix)top_3d_laser" parent="$(arg prefix)base_link" gpu="$(arg gpu)">
-			<origin xyz="-0.11808 0.0 0.38509" rpy="0 0 0"/>
-		</xacro:sensor_rs_helios_16p>
-		<!-- ptz camera -->
-		<!--xacro:sensor_axis prefix="$(arg prefix)front_ptz_camera" parent="$(arg prefix)base_link">
-			<origin xyz="0.19 0 0.26" rpy="0 ${15*PI/180} 0"/>
-		</xacro:sensor_axis-->
-	  <!-- RGBD -->
-	  <xacro:sensor_orbbec_astra prefix="$(arg prefix)front_rgbd_camera" parent="$(arg prefix)base_link" prefix_topic="front_rgbd_camera">
+	<!-- Wheel parameters -->
+	<xacro:property name="wheel_offset_x" value="0.229" />    <!-- x,y,z in translation from base_link to the center of the wheel -->
+	<xacro:property name="wheel_offset_y" value="0.235" />
+	<xacro:property name="wheel_offset_z" value="0.0" />
+	<!-- Here we create the robot using the xacro:macro imported at the beggining of this file -->
+   	<xacro:summit_xl robot_id="$(arg robot_id)" publish_bf="true" hq="true" kinematics="$(arg kinematics)"/>
+	<!-- Custom Sensors -->
+	<!-- IMU -->
+	<!-- <xacro:sensor_imu prefix="$(arg prefix)imu" parent="$(arg prefix)base_link" topic="imu/data_raw">
+		<origin xyz="0.0385 0.132 0.158" rpy="0 0 0"/>
+	</xacro:sensor_imu> -->
+	<!-- 3d laser -->
+	<!-- <xacro:sensor_rs_helios_16p prefix="$(arg prefix)top_3d_laser" parent="$(arg prefix)base_link" gpu="$(arg gpu)">
+		<origin xyz="-0.11808 0.0 0.38509" rpy="0 0 0"/>
+	</xacro:sensor_rs_helios_16p> -->
+	<!-- ptz camera -->
+	<!-- <xacro:sensor_axis_m5525 prefix="$(arg prefix)front_ptz_camera" parent="$(arg prefix)base_link">
+		<origin xyz="0.19 0 0.26" rpy="0 ${15*PI/180} 0"/>
+	</xacro:sensor_axis_m5525> -->
+	<!-- RGBD -->
+	<!-- <xacro:sensor_orbbec_astra prefix="$(arg prefix)front_rgbd_camera" parent="$(arg prefix)base_link">
 			<origin xyz="0.324 0.012 0.172" rpy="0 0 0"/>
-		</xacro:sensor_orbbec_astra>
-	  <!-- GPS -->
-	  <xacro:sensor_gps_with_mast prefix="$(arg prefix)gps" parent="$(arg prefix)base_link" gps_latitude="$(arg gps_latitude)" gps_longitude="$(arg gps_longitude)" update_rate="5">
+		</xacro:sensor_orbbec_astra> -->
+	<!-- GPS -->
+	<!-- <xacro:sensor_gps_with_mast prefix="$(arg prefix)gps" parent="$(arg prefix)base_link" gps_latitude="$(arg gps_latitude)" gps_longitude="$(arg gps_longitude)" update_rate="5">
 			<origin xyz="-0.22528 0.095 0.275" rpy="0 0 0"/>
-		</xacro:sensor_gps_with_mast>
-	  <!--Antenna-->
-	  <xacro:structure_mastil_teltonika prefix="$(arg prefix)antenna" parent="$(arg prefix)base_link">
+		</xacro:sensor_gps_with_mast> -->
+	<!--Antenna-->
+	<!-- <xacro:structure_mastil_teltonika prefix="$(arg prefix)antenna" parent="$(arg prefix)base_link">
 			<origin xyz="-0.22528 -0.095 0.23325" rpy="0 0 0"/>
-		</xacro:structure_mastil_teltonika>
-	  <!-- Gazebo ros control pluggins -->
-      <xacro:ros_control/>
-	  <xacro:if value="$(arg ros_planar_move_plugin)">
-		<xacro:if value="${kinematics == 'omni' or kinematics == 'omni_4w'}">
-			<xacro:omni_steering prefix="$(arg prefix)" publish_tf="true" force_based="$(arg ros_planar_move_plugin_force_based)"/>
-		</xacro:if>
-		<xacro:if value="${kinematics == 'skid' or kinematics == 'skid_4w'}">
-			<xacro:skid_steering prefix="$(arg prefix)" publish_tf="true" force_based="$(arg ros_planar_move_plugin_force_based)"/>
-		</xacro:if>
-	  </xacro:if>
-   </xacro:macro>
-   <xacro:summit_xl prefix="$(arg prefix)" publish_bf="true" hq="true" kinematics="$(arg kinematics)"/>
+		</xacro:structure_mastil_teltonika> -->
 </robot>
