Commit message: urdf/rbsherkan_rocker: Set as fixed joint

File: urdf/structures/rbsherkan_chassis/rbsherkan_rocker.urdf.xacro (robot description, xacro)
@@ -5,11 +5,9 @@
     <xacro:include filename="$(find robot_description)/urdf/wheels/rubber_wheel/rubber_wheel_150.urdf.xacro" />
     <!-- Base link -->
-    <joint name="${prefix}rocker_joint" type="revolute">
+    <joint name="${prefix}rocker_joint" type="fixed">
       <xacro:insert_block name="origin" />
       <parent link="${parent}"/>
       <child link="${prefix}rocker_link"/>
       <axis xyz="0 1 0" />
-      <limit effort="100" lower="-0.35" upper="0.35" velocity="100" />
-      <dynamics damping="0.0" friction="0.95"/>
     </joint>
     <link name="${prefix}rocker_link">
