Commit message: Optimize summit_hm model meshes

File: urdf/bases/summit_hm_base.urdf.xacro (robot description, xacro)
@@ -50,5 +50,5 @@
 			<xacro:unless value="${hq}">
 			<geometry>
-				<mesh filename="package://robot_description/meshes/bases/summit_hm_body.stl"/>
+				<mesh filename="package://robot_description/meshes/bases/summit_hm_body.dae"/>
 			</geometry>
 			</xacro:unless>
@@ -60,8 +60,12 @@
 			<origin xyz="0 0 0" rpy="0 0 0 " />
 			<geometry>
-				<mesh filename="package://robot_description/meshes/bases/summit_hm_body.dae"/>
+				<mesh filename="package://robot_description/meshes/bases/summit_hm_body.stl"/>
 			</geometry>
 		</collision>
 		</link>
+		<gazebo reference="${prefix}base_link">
+			<material>Gazebo/Gray</material>
+			<turnGravityOff>false</turnGravityOff>
+		</gazebo>
 		<!-- DOCKING CONTACTS -->
 		<joint name="${prefix}base_docking_joint" type="fixed">

File: urdf/structures/summit_hm/summit_hm_structure.xacro (robot description, xacro)
@@ -21,5 +21,5 @@
         </material>
 	      <geometry>
-	        <mesh filename="package://${mesh_file}.stl"/>
+	        <mesh filename="package://${mesh_file}.dae"/>
 	      </geometry>
 	    </visual>
@@ -27,5 +27,5 @@
 	      <origin rpy="0 0 0" xyz="0 0 0"/>
 	      <geometry>
-	        <mesh filename="package://${mesh_file}.dae"/>
+	        <mesh filename="package://${mesh_file}.stl"/>
 	      </geometry>
 	    </collision>

File: urdf/wheels/rubber_wheel/rubber_wheel.urdf.xacro (robot description, xacro)
@@ -45,8 +45,8 @@
         <geometry>
           <xacro:if value="${reflect}">
-							<mesh filename="package://${mesh_file_left}.dae" />
+							<mesh filename="package://${mesh_file_left}.stl" />
 						</xacro:if>
 						<xacro:unless value="${reflect}">
-							<mesh filename="package://${mesh_file_right}.dae" />
+							<mesh filename="package://${mesh_file_right}.stl" />
           </xacro:unless>
         </geometry>
@@ -69,4 +69,8 @@
       </actuator>
      </transmission>
+    <gazebo reference="${prefix}_wheel">
+			<material>Gazebo/Black</material>
+			<turnGravityOff>false</turnGravityOff>
+		</gazebo>
   </xacro:macro>
 </robot>
