Commit message: Standarize robot_id and eliminate prefix

File: urdf/bases/rb_theron_base.urdf.xacro (robot description, xacro)
@@ -25,26 +25,26 @@
 	<!-- Robots Elements -->
 	<!-- *************** -->
-  <xacro:macro name="rb_theron_base" params="prefix hq use_sim">
+  <xacro:macro name="rb_theron_base" params="robot_id hq use_sim">
     <!-- rb_theron base -->
-  	<xacro:rb_theron_base_v4 prefix="${prefix}" publish_bf="true" hq="${hq}" />
-    <xacro:gazebo_colors prefix="${prefix}"/>
+  	<xacro:rb_theron_base_v4 robot_id="${robot_id}" publish_bf="true" hq="${hq}" />
+    <xacro:gazebo_colors robot_id="${robot_id}"/>
   	<!-- WHEELS -->
-  	<xacro:rubber_wheel prefix="${prefix}right" parent="${prefix}base_link" hq="${hq}">
+  	<xacro:rubber_wheel robot_id="${robot_id}_right" parent="${robot_id}_base_link" hq="${hq}">
   		<origin xyz="${wheel_offset_x} ${-wheel_offset_y} ${wheel_offset_z}" rpy="0 0 0"/>
   	</xacro:rubber_wheel>
-  	<xacro:rubber_wheel prefix="${prefix}left" parent="${prefix}base_link" hq="${hq}">
+  	<xacro:rubber_wheel robot_id="${robot_id}_left" parent="${robot_id}_base_link" hq="${hq}">
   		<origin xyz="${wheel_offset_x} ${wheel_offset_y} ${wheel_offset_z}" rpy="0 0 0"/>
   	</xacro:rubber_wheel>
 <!-- Castor wheels-->
-	<xacro:caster prefix="${prefix}front_left" parent="${prefix}base_link" hq="${hq}" use_sim="$(arg use_sim)">
+	<xacro:caster robot_id="${robot_id}_front_left" parent="${robot_id}_base_link" hq="${hq}" use_sim="$(arg use_sim)">
 		<origin xyz="0.235 0.1825 0.0448" rpy="0 0 0"/>
 	</xacro:caster>
-	<xacro:caster prefix="${prefix}front_right" parent="${prefix}base_link" hq="${hq}" use_sim="$(arg use_sim)">
+	<xacro:caster robot_id="${robot_id}_front_right" parent="${robot_id}_base_link" hq="${hq}" use_sim="$(arg use_sim)">
 		<origin xyz="0.235 -0.1825 0.0448" rpy="0 0 0"/>
 	</xacro:caster>
-	<xacro:caster prefix="${prefix}rear_left" parent="${prefix}base_link" hq="${hq}" use_sim="$(arg use_sim)">
+	<xacro:caster robot_id="${robot_id}_rear_left" parent="${robot_id}_base_link" hq="${hq}" use_sim="$(arg use_sim)">
 		<origin xyz="-0.235 0.1825 0.0448" rpy="0 0 0"/>
 	</xacro:caster>
-	<xacro:caster prefix="${prefix}rear_right" parent="${prefix}base_link" hq="${hq}" use_sim="$(arg use_sim)">
+	<xacro:caster robot_id="${robot_id}_rear_right" parent="${robot_id}_base_link" hq="${hq}" use_sim="$(arg use_sim)">
 		<origin xyz="-0.235 -0.1825 0.0448" rpy="0 0 0"/>
 	</xacro:caster>

File: urdf/bases/rb_theron_base_v4.urdf.xacro (robot description, xacro)
@@ -2,5 +2,5 @@
 <robot name="rb_theron_v4" xmlns:xacro="http://wiki.ros.org/xacro">
   <xacro:include filename="$(find robot_description)/urdf/bases/gazebo/rb_theron_base.gazebo.xacro" />
-  <xacro:macro name="rb_theron_base_v4" params="prefix publish_bf hq">
+  <xacro:macro name="rb_theron_base_v4" params="robot_id publish_bf hq">
   <!-- Robot mechanical and motor parameters -->
   <xacro:property name="PI" value="3.1415926535897931"/>
@@ -8,5 +8,5 @@
 	<!-- BASE FOOTPRINT -->
 	  <xacro:if value="${publish_bf}">
-		<link name="${prefix}base_footprint">
+		<link name="${robot_id}_base_footprint">
 		  <visual>
 			  <origin xyz="0 0 0" rpy="0 0 0" />
@@ -16,12 +16,12 @@
 		  </visual>
 		</link>
-		<joint name="${prefix}base_footprint_joint" type="fixed">
+		<joint name="${robot_id}_base_footprint_joint" type="fixed">
 		  <origin xyz="0 0 ${wheel_radius}" rpy="0 0 0" /> <!-- ${wheel_radius} property must be defined inside wheel description -->
-		  <parent link="${prefix}base_footprint"/>
-		  <child link="${prefix}base_link" />
+		  <parent link="${robot_id}_base_footprint"/>
+		  <child link="${robot_id}_base_link" />
 		</joint>
 	  </xacro:if>
   <!-- BASE_LINK -->
-  <link name="${prefix}base_link">
+  <link name="${robot_id}_base_link">
     <inertial>
       <mass value="45.0" />
@@ -52,9 +52,9 @@
     </collision>
   </link>
-  <gazebo reference="${prefix}base_link">
+  <gazebo reference="${robot_id}_base_link">
     <material>Gazebo/Black</material>
   </gazebo>
   <!-- CHAPAS INOX TAPAS -->
-  <!--link name="${prefix}base_chapa">
+  <!--link name="${robot_id}_base_chapa">
   <visual>
     <origin xyz="0 0 0" rpy="0 0 0" />
@@ -67,11 +67,11 @@
     </visual>
   </link-->
-  <!--joint name="${prefix}base_tapa_joint" type="fixed">
+  <!--joint name="${robot_id}_base_tapa_joint" type="fixed">
     <origin xyz="0.0 0 0.38062" rpy="0 0 0" />
-    <parent link="${prefix}base_link"/>
-    <child link="${prefix}base_chapa" />
+    <parent link="${robot_id}_base_link"/>
+    <child link="${robot_id}_base_chapa" />
   </joint-->
   <!-- LOGO ROBOTNIK IZQUIERDO >
-  <link name="${prefix}base_logo_left">
+  <link name="${robot_id}_base_logo_left">
   <visual>
     <origin xyz="0 0 0" rpy="0 0 0" />
@@ -84,11 +84,11 @@
     </visual>
   </link>
-  <joint name="${prefix}base_logo_left_joint" type="fixed">
+  <joint name="${robot_id}_base_logo_left_joint" type="fixed">
     <origin xyz="0.0 0.28931 0.29062" rpy="0 0 0" />
-    <parent link="${prefix}base_link"/>
-    <child link="${prefix}base_logo_left" />
+    <parent link="${robot_id}_base_link"/>
+    <child link="${robot_id}_base_logo_left" />
   </joint-->
   <!-- LOGO ROBOTNIK DERECHO >
-  <link name="${prefix}base_logo_right">
+  <link name="${robot_id}_base_logo_right">
   <visual>
     <origin xyz="0 0 0" rpy="0 0 0" />
@@ -101,11 +101,11 @@
     </visual>
   </link>
-  <joint name="${prefix}base_logo_right_joint" type="fixed">
+  <joint name="${robot_id}_base_logo_right_joint" type="fixed">
     <origin xyz="0.0 -0.28931 0.29062" rpy="0 0 ${PI}" />
-    <parent link="${prefix}base_link"/>
-    <child link="${prefix}base_logo_right" />
+    <parent link="${robot_id}_base_link"/>
+    <child link="${robot_id}_base_logo_right" />
   </joint-->
   <!-- LOGO ROBOTNIK FRONTAL >
-  <link name="${prefix}base_logo_front">
+  <link name="${robot_id}_base_logo_front">
   <visual>
     <origin xyz="0 0 0" rpy="0 0 0" />
@@ -118,11 +118,11 @@
     </visual>
   </link>
-  <joint name="${prefix}base_logo_front_joint" type="fixed">
+  <joint name="${robot_id}_base_logo_front_joint" type="fixed">
     <origin xyz="0.345 0.0 0.0" rpy="0 0 ${-PI/2}" />
-    <parent link="${prefix}base_link"/>
-    <child link="${prefix}base_logo_front" />
+    <parent link="${robot_id}_base_link"/>
+    <child link="${robot_id}_base_logo_front" />
   </joint-->
   <!-- LOGO ROBOTNIK TRASERO >
-  <link name="${prefix}base_logo_rear">
+  <link name="${robot_id}_base_logo_rear">
   <visual>
     <origin xyz="0 0 0" rpy="0 0 0" />
@@ -135,16 +135,16 @@
     </visual>
   </link>
-  <joint name="${prefix}base_logo_rear_joint" type="fixed">
+  <joint name="${robot_id}_base_logo_rear_joint" type="fixed">
     <origin xyz="-0.345 0.0 0.0" rpy="0 0 ${PI/2}" />
-    <parent link="${prefix}base_link"/>
-    <child link="${prefix}base_logo_rear" />
+    <parent link="${robot_id}_base_link"/>
+    <child link="${robot_id}_base_logo_rear" />
   </joint-->
    <!-- DOCKING CONTACT -->
-    <link name="${prefix}base_docking_contact">
+    <link name="${robot_id}_base_docking_contact">
     </link>
-    <joint name="${prefix}base_docking_joint" type="fixed">
+    <joint name="${robot_id}_base_docking_joint" type="fixed">
       <origin xyz="0.35 0 0.09" rpy="0 0 0" />
-      <parent link="${prefix}base_link"/>
-      <child link="${prefix}base_docking_contact" />
+      <parent link="${robot_id}_base_link"/>
+      <child link="${robot_id}_base_docking_contact" />
     </joint>
   </xacro:macro>

File: urdf/bases/summit_xl_base.urdf.xacro (robot description, xacro)
@@ -2,5 +2,5 @@
 <robot name="summit_xl" xmlns:xacro="http://wiki.ros.org/xacro">
   <xacro:include filename="$(find robot_description)/urdf/bases/gazebo/summit_xl_base.gazebo.xacro" />
-  <xacro:macro name="summit_xl_base" params="prefix publish_bf hq">
+  <xacro:macro name="summit_xl_base" params="robot_id publish_bf hq">
 	  <!-- Robot mechanical and motor parameters -->
 	  <xacro:property name="PI" value="3.1415926535897931"/>
@@ -8,5 +8,5 @@
 	  <!-- BASE FOOTPRINT -->
 	  <xacro:if value="${publish_bf}">
-		<link name="${prefix}base_footprint">
+		<link name="${robot_id}_base_footprint">
 		  <visual>
 			  <origin xyz="0 0 0" rpy="0 0 0" />
@@ -16,12 +16,12 @@
 		  </visual>
 		</link>
-		<joint name="${prefix}base_footprint_joint" type="fixed">
+		<joint name="${robot_id}_base_footprint_joint" type="fixed">
 		  <origin xyz="0 0 ${wheel_radius}" rpy="0 0 0" /> <!-- ${wheel_radius} property must be defined inside wheel description -->
-		  <parent link="${prefix}base_footprint"/>
-		  <child link="${prefix}base_link" />
+		  <parent link="${robot_id}_base_footprint"/>
+		  <child link="${robot_id}_base_link" />
 		</joint>
 	  </xacro:if>
 	  <!-- BASE_LINK -->
-	  <link name="${prefix}base_link">
+	  <link name="${robot_id}_base_link">
 		<inertial>
 		  <mass value="25.0" />
@@ -53,11 +53,11 @@
 	  </link>
 		<!-- DOCKING CONTACTS -->
-		<joint name="${prefix}base_docking_joint" type="fixed">
+		<joint name="${robot_id}_base_docking_joint" type="fixed">
 			<origin xyz="0.284 0.012 0.068" rpy="0 0 0 " />
-			<parent link="${prefix}base_link"/>
-			<child link="${prefix}base_docking_contact_link" />
+			<parent link="${robot_id}_base_link"/>
+			<child link="${robot_id}_base_docking_contact_link" />
 		</joint>
 		<!-- DOCKING LINK -->
-		<link name="${prefix}base_docking_contact_link" />
+		<link name="${robot_id}_base_docking_contact_link" />
   </xacro:macro>
 </robot>

File: urdf/wheels/caster_wheel/rb_theron_caster.urdf.xacro (robot description, xacro)
@@ -18,10 +18,10 @@
               izz="${m*r*r/2}" />
   </xacro:macro>
-  <xacro:macro name="caster" params="prefix parent *origin hq use_sim">
+  <xacro:macro name="caster" params="robot_id parent *origin hq use_sim">
   <!--CASTER SUPPORT -->
   <xacro:if value="${use_sim}">
-    <joint name="${prefix}joint_support" type="continuous">
+    <joint name="${robot_id}_joint_support" type="continuous">
       <parent link="${parent}"/>
-      <child link="${prefix}_support"/>
+      <child link="${robot_id}_support"/>
       <xacro:insert_block name="origin" />
       <axis xyz="0 0 1" rpy="0 ${M_PI} 0" />
@@ -32,7 +32,7 @@
   </xacro:if>
   <xacro:unless value="${use_sim}">
-    <joint name="${prefix}joint_support" type="fixed">
+    <joint name="${robot_id}_joint_support" type="fixed">
         <parent link="${parent}"/>
-        <child link="${prefix}_support"/>
+        <child link="${robot_id}_support"/>
         <xacro:insert_block name="origin" />
         <axis xyz="0 0 1" rpy="0 ${M_PI} 0" />
@@ -42,5 +42,5 @@
       </joint>
   </xacro:unless>
-    <link name="${prefix}_support">
+    <link name="${robot_id}_support">
       <visual>
         <origin xyz="0 0 0" rpy="0 0 0" />
@@ -62,14 +62,14 @@
     </link>
   <!--CASTER WHEEL -->
-  <!-- xacro:caster_wheel prefix="${prefix}" parent="${prefix}_support" hq="${hq}" -->
-  <xacro:caster_wheel prefix="${prefix}" parent="${prefix}_support" hq="${hq}" use_sim="$(arg use_sim)">
+  <!-- xacro:caster_wheel robot_id="${robot_id}" parent="${robot_id}_support" hq="${hq}" -->
+  <xacro:caster_wheel robot_id="${robot_id}" parent="${robot_id}_support" hq="${hq}" use_sim="$(arg use_sim)">
 		<origin xyz="${caster_wheel_offset_x} ${caster_wheel_offset_y} ${caster_wheel_offset_z}" rpy="0 0 0"/>
    </xacro:caster_wheel>
  </xacro:macro>
- <xacro:macro name="caster_wheel" params="prefix parent *origin hq use_sim">
+ <xacro:macro name="caster_wheel" params="robot_id parent *origin hq use_sim">
   <xacro:if value="${use_sim}">
-    <joint name="${prefix}joint_wheel" type="continuous">
+    <joint name="${robot_id}_joint_wheel" type="continuous">
       <parent link="${parent}"/>
-      <child link="${prefix}_wheel"/>
+      <child link="${robot_id}_wheel"/>
       <insert_block name="origin" />
       <axis xyz="0 1 0" rpy="0 0 0" />
@@ -79,7 +79,7 @@
   </xacro:if>
   <xacro:unless value="${use_sim}">
-     <joint name="${prefix}joint_wheel" type="fixed">
+     <joint name="${robot_id}_joint_wheel" type="fixed">
        <parent link="${parent}"/>
-       <child link="${prefix}_wheel"/>
+       <child link="${robot_id}_wheel"/>
        <insert_block name="origin" />
        <axis xyz="0 1 0" rpy="0 0 0" />
@@ -88,5 +88,5 @@
     </joint>
   </xacro:unless>
-    <link name="${prefix}_wheel">
+    <link name="${robot_id}_wheel">
       <visual>
         <!-- HIGH RESOLUTION WHEELS -->
@@ -126,20 +126,20 @@
   <!-- Transmission is important to link the joints and the controller-->
   <xacro:if value="${use_sim}">
-    <transmission name="${prefix}_support_joint_trans">
+    <transmission name="${robot_id}_support_joint_trans">
       <type>transmission_interface/SimpleTransmission</type>
-      <joint name="${prefix}joint_support">
+      <joint name="${robot_id}_joint_support">
           <hardwareInterface>hardware_interface/EffortJointInterface</hardwareInterface>
       </joint>
-      <actuator name="${prefix}_support_joint_motor">
+      <actuator name="${robot_id}_support_joint_motor">
         <mechanicalReduction>1</mechanicalReduction>
       	<motorTorqueConstant>1</motorTorqueConstant>
       </actuator>
     </transmission>
-    <transmission name="${prefix}_wheel_joint_trans">
+    <transmission name="${robot_id}_wheel_joint_trans">
       <type>transmission_interface/SimpleTransmission</type>
-      <joint name="${prefix}joint_wheel">
+      <joint name="${robot_id}_joint_wheel">
           <hardwareInterface>hardware_interface/EffortJointInterface</hardwareInterface>
       </joint>
-      <actuator name="${prefix}_wheel_joint_motor">
+      <actuator name="${robot_id}_wheel_joint_motor">
         <mechanicalReduction>1</mechanicalReduction>
 		<motorTorqueConstant>1</motorTorqueConstant>
@@ -147,5 +147,5 @@
     </transmission>
   </xacro:if>
-    <gazebo reference="${prefix}_support">
+    <gazebo reference="${robot_id}_support">
 			<mu1 value="5.0"/>
 			<mu2 value="0.5"/>
@@ -155,5 +155,5 @@
       <turnGravityOff>false</turnGravityOff>
     </gazebo>
-     <gazebo reference="${prefix}_wheel">
+     <gazebo reference="${robot_id}_wheel">
 			<mu1 value="100.0"/>
 			<mu2 value="100.0"/>

File: urdf/wheels/omni_wheel/omni_wheel.urdf.xacro (robot description, xacro)
@@ -11,8 +11,8 @@
               izz="${m*(3*r*r+h*h)/12}" />
   </xacro:macro>
-  <xacro:macro name="omni_wheel" params="prefix parent *origin reflect hq">
-    <joint name="${prefix}_wheel_joint" type="continuous">
+  <xacro:macro name="omni_wheel" params="robot_id parent *origin reflect hq">
+    <joint name="${robot_id}_wheel_joint" type="continuous">
       <parent link="${parent}"/>
-      <child link="${prefix}_wheel_link"/>
+      <child link="${robot_id}_wheel_link"/>
       <xacro:insert_block name="origin" />
       <axis xyz="0 1 0" rpy="0 0 0" />
@@ -20,5 +20,5 @@
       <joint_properties damping="1.0" friction="1.0"/>
     </joint>
-    <link name="${prefix}_wheel_link">
+    <link name="${robot_id}_wheel_link">
       <visual>
         <xacro:if value="${hq}">
@@ -68,14 +68,14 @@
     </link>
     <!-- Transmission is important to link the joints and the controller (see summit_xl_control/config/summit_xl_control.yaml)-->
-    <!-- <transmission name="${prefix}_wheel_joint_trans">
+    <!-- <transmission name="${robot_id}_wheel_joint_trans">
       <type>transmission_interface/SimpleTransmission</type>
-      <joint name="${prefix}_wheel_joint" >
+      <joint name="${robot_id}_wheel_joint" >
         <hardwareInterface>hardware_interface/VelocityJointInterface</hardwareInterface>
       </joint>
-      <actuator name="${prefix}_wheel_joint_motor">
+      <actuator name="${robot_id}_wheel_joint_motor">
          <mechanicalReduction>1</mechanicalReduction>
       </actuator>
     </transmission> -->
-    <gazebo reference="${prefix}_wheel_link">
+    <gazebo reference="${robot_id}_wheel_link">
       <mu1>0.90</mu1>
       <mu2>0.85</mu2>

File: urdf/wheels/rubber_wheel/rubber_wheel.urdf.xacro (robot description, xacro)
@@ -7,10 +7,10 @@
               izz="${m*(3*r*r+h*h)/12}" />
   </xacro:macro>
-  <xacro:macro name="rubber_wheel" params="prefix parent *origin *axis reflect hq rubber_wheel_radius:=0.11 rubber_wheel_width:=0.15 rubber_wheel_mass:=6.5
+  <xacro:macro name="rubber_wheel" params="robot_id parent *origin *axis reflect hq rubber_wheel_radius:=0.11 rubber_wheel_width:=0.15 rubber_wheel_mass:=6.5
                                           mesh_file:=robot_description/meshes/wheels/rubber_wheel/rubber_wheel_right">
 <!--WHEEL TIRE -->
-    <joint name="${prefix}_wheel_joint" type="continuous">
+    <joint name="${robot_id}_wheel_joint" type="continuous">
       <parent link="${parent}"/>
-      <child link="${prefix}_wheel"/>
+      <child link="${robot_id}_wheel"/>
       <xacro:insert_block name="origin" />
       <xacro:insert_block name="axis" />
@@ -18,5 +18,5 @@
       <joint_properties damping="0.0" friction="0.0"/>
     </joint>
-    <link name="${prefix}_wheel">
+    <link name="${robot_id}_wheel">
       <visual>
         <!-- HIGH RESOLUTION WHEELS -->
@@ -48,5 +48,5 @@
           </xacro:if>
           <geometry>
-						<mesh filename="package://${mesh_file}.stl" />
+						<mesh filename="package://${mesh_file}.dae" />
         </geometry>
       </collision>
@@ -58,16 +58,21 @@
     </link>
     <!-- Transmission is important to link the joints and the controller (see summit_xl_control/config/summit_xl_control.yaml)-->
-    <transmission name="${prefix}_wheel_joint_trans">
+    <transmission name="${robot_id}_wheel_joint_trans">
       <type>transmission_interface/SimpleTransmission</type>
-      <joint name="${prefix}_wheel_joint">
+      <joint name="${robot_id}_wheel_joint">
         <hardwareInterface>hardware_interface/VelocityJointInterface</hardwareInterface>
       </joint>
-      <actuator name="${prefix}_wheel_joint_motor">
+      <actuator name="${robot_id}_wheel_joint_motor">
         <mechanicalReduction>1</mechanicalReduction>
         <motorTorqueConstant>20</motorTorqueConstant>
       </actuator>
      </transmission>
-    <gazebo reference="${prefix}_wheel">
-			<material>Gazebo/Black</material>
+    <gazebo reference="${robot_id}_wheel">
+			<!-- <material>Gazebo/Black</material> -->
+      <mu1 value="1.0"/>
+			<mu2 value="1.0"/>
+			<kp value="10000000.0" />
+			<kd value="1.0" />
+			<fdir1 value="1 0 0"/>
 			<turnGravityOff>false</turnGravityOff>
 		</gazebo>
