Commit message: Basic robots checked, change repository structure

File: urdf/bases/gazebo/rbvogui_base.gazebo.xacro (robot description, xacro)
@@ -1,51 +1,7 @@
 <?xml version="1.0"?>
 <robot xmlns:xacro="http://wiki.ros.org/xacro">
-    <!-- ros control plugin -->
-    <xacro:macro name="ros_control">
-        <gazebo>
-            <plugin name="ros_control" filename="libgazebo_ros_control.so">
-                <!--<robotNamespace>/summit_xl</robotNamespace>-->
-                <robotParam>robot_description</robotParam>
-                <controlPeriod>0.001</controlPeriod>
-                <robotSimType>gazebo_ros_control/DefaultRobotHWSim</robotSimType>
-                <legacyModeNS>true</legacyModeNS>
-            </plugin>
-        </gazebo>
-    </xacro:macro>
-    <xacro:macro name="omni_steering">
-        <gazebo>
-            <plugin name="omni_steering" filename="libgazebo_ros_planar_move.so">
-                <robotNamespace>/robot</robotNamespace>
-                <commandTopic>robotnik_base_control/cmd_vel</commandTopic>
-                <odometryTopic>robotnik_base_control/odom</odometryTopic>
-                <odometryFrame>odom</odometryFrame>
-                <odometryRate>20.0</odometryRate>
-                <robotBaseFrame>base_footprint</robotBaseFrame>
-            </plugin>
-          </gazebo>
-    </xacro:macro>
-    <xacro:macro name="omni_drive_ackermann">
-        <gazebo>
-            <plugin name="omni_drive_ackermann" filename="libomnidrive_ackermann_plugin.so">
-                <!--<robotNamespace>/rbvogui</robotNamespace>-->
-                <!--<robotParam>robot_description</robotParam>-->
-                <broadcastTF>1</broadcastTF>
-                <wheelDiameter>0.220</wheelDiameter>
-                <wheelBase>0.858</wheelBase>
-                <trackWidth>0.454</trackWidth>
-                <wheelTorque>44.2</wheelTorque>
-                <motorWheelTorque>15.0</motorWheelTorque>
-                <commandTopic>cmd_vel</commandTopic>  <!-- TODO: review topics -->
-                <odometryTopic>odom</odometryTopic>
-                <odometryFrame>odom</odometryFrame>
-                <odometrySource>encoder</odometrySource>
-                <robotBaseFrame>base_footprint</robotBaseFrame>
-                <updateRate>100.0</updateRate>
-            </plugin>
-        </gazebo>
-    </xacro:macro>
    <!-- not used in 6w -->
-    <xacro:macro name="gazebo_color_base_link" params="prefix">
-      <gazebo reference="${prefix}base_link">
+    <xacro:macro name="gazebo_color_base_link" params="robot_id">
+      <gazebo reference="${robot_id}_base_link">
         <visual>
           <material>
@@ -58,6 +14,6 @@
       </gazebo>
     </xacro:macro>
-    <xacro:macro name="gazebo_color_chassis_link" params="prefix">
-      <gazebo reference="${prefix}chassis_link">
+    <xacro:macro name="gazebo_color_chassis_link" params="robot_id">
+      <gazebo reference="${robot_id}_chassis_link">
         <visual>
           <material>
@@ -70,6 +26,6 @@
       </gazebo>
     </xacro:macro>
-    <xacro:macro name="gazebo_color_logo_link" params="prefix">
-      <gazebo reference="${prefix}base_logos_link">
+    <xacro:macro name="gazebo_color_logo_link" params="robot_id">
+      <gazebo reference="${robot_id}_base_logos_link">
         <visual>
           <material>
@@ -82,6 +38,6 @@
       </gazebo>
     </xacro:macro>
-    <xacro:macro name="gazebo_color_battery_link" params="prefix">
-      <gazebo reference="${prefix}battery_link">
+    <xacro:macro name="gazebo_color_battery_link" params="robot_id">
+      <gazebo reference="${robot_id}_battery_link">
         <visual>
           <material>
@@ -94,6 +50,6 @@
       </gazebo>
     </xacro:macro>
-    <xacro:macro name="gazebo_color_contactors_link" params="prefix">
-      <gazebo reference="${prefix}contactors_link">
+    <xacro:macro name="gazebo_color_contactors_link" params="robot_id">
+      <gazebo reference="${robot_id}_contactors_link">
         <visual>
           <material>
@@ -106,6 +62,6 @@
       </gazebo>
     </xacro:macro>
-    <xacro:macro name="gazebo_color_leds_link" params="prefix">
-      <gazebo reference="${prefix}leds_link">
+    <xacro:macro name="gazebo_color_leds_link" params="robot_id">
+      <gazebo reference="${robot_id}_leds_link">
         <visual>
           <material>

File: urdf/wheels/fixed_wheel/fixed_wheel.urdf.xacro (robot description, xacro)
@@ -1,6 +1,6 @@
 <?xml version="1.0"?>
 <robot xmlns:xacro="http://www.ros.org/wiki/xacro">
-  <xacro:include filename="$(find robot_description)/urdf/wheels/rubber_wheel/gazebo/rbvogui_wheel.gazebo.xacro" />
-  <xacro:include filename="$(find robot_description)/urdf/wheels/rubber_wheel/rbvogui_rubber_wheel.urdf.xacro" />
+  <xacro:include filename="$(find robot_description)/urdf/wheels/wheel.gazebo.xacro" />
+  <xacro:include filename="$(find robot_description)/urdf/wheels/rubber_wheel.urdf.xacro" />
   <xacro:property name="M_PI" value="3.1415926535897931" />
   <!-- Wheels -->
@@ -23,6 +23,4 @@
   </xacro:macro>
   <xacro:macro name="fixed_wheel" params="prefix parent *origin reflect hq">
-    <!-- TODO: check reflect parameter -->
-    <!--MOTOR WHEEL -->
     <joint name="${prefix}fixed_wheel_joint" type="fixed">
       <parent link="${parent}"/>
@@ -30,5 +28,4 @@
       <xacro:insert_block name="origin" />
       <axis xyz="0 0 1" rpy="0 0 0" />
-      <!-- limit effort="${steer_joint_effort_limit}" velocity="${steer_joint_velocity_limit}" lower="-1.5708" upper="1.5708" / -->
       <limit effort="${steer_joint_effort_limit}" velocity="${steer_joint_velocity_limit}" lower="-3.00" upper="3.00"/>
       <joint_properties damping="${steer_joint_damping}" friction="${steer_joint_friction}"/>
@@ -45,5 +42,5 @@
           </xacro:unless>
           <geometry>
-            <mesh filename="package://robot_description/meshes/wheels/rubber_wheel/mw_frame.stl" />
+            <mesh filename="package://robot_description/meshes/wheels/mw_frame.stl" />
           </geometry>
         </xacro:if>
@@ -57,5 +54,5 @@
           </xacro:unless>
           <geometry>
-            <mesh filename="package://robot_description/meshes/wheels/rubber_wheel/mw_frame.stl" />
+            <mesh filename="package://robot_description/meshes/wheels/mw_frame.stl" />
           </geometry>
         </xacro:unless>
@@ -72,5 +69,5 @@
         </xacro:unless>
         <geometry>
-          <mesh filename="package://robot_description/meshes/wheels/rubber_wheel/mw_frame.stl" />
+          <mesh filename="package://robot_description/meshes/wheels/mw_frame.stl" />
         </geometry>
       </collision>

File: urdf/wheels/omni_wheel/omni_wheel.urdf.xacro (robot description, xacro)
@@ -26,10 +26,10 @@
           <xacro:if value="${reflect}">
             <geometry>
-              <mesh filename="package://robot_description/meshes/wheels/omni_wheel/wheel_omni_4inch.dae" />
+              <mesh filename="package://robot_description/meshes/wheels/omni_wheel/omni_wheel_1.dae" />
             </geometry>
           </xacro:if>
           <xacro:unless value="${reflect}">
             <geometry>
-              <mesh filename="package://robot_description/meshes/wheels/omni_wheel/wheel_omni_4inch.dae" />
+              <mesh filename="package://robot_description/meshes/wheels/omni_wheel/omni_wheel_2.dae" />
             </geometry>
 		  </xacro:unless>
@@ -48,15 +48,5 @@
 				<origin xyz="0 0 0" rpy="${PI/2} 0 0" />
         <geometry>
-          <!--sphere radius="${omni_wheel_radius}" /-->
-<!--
-          <xacro:if value="${reflect}">
-              <mesh filename="package://robot_description/meshes/wheels/omni_wheel/omni_wheel_1.dae" />
-          </xacro:if>
-          <xacro:unless value="${reflect}">
-              <mesh filename="package://robot_description/meshes/wheels/omni_wheel/omni_wheel_2.dae" />
-					</xacro:unless>
--->
 					<cylinder length="${omni_wheel_height}" radius="${omni_wheel_radius}" />
-					<!-- sphere radius="${omni_wheel_radius}"/-->
         </geometry>
       </collision>
@@ -67,14 +57,4 @@
       </inertial>
     </link>
-    <!-- Transmission is important to link the joints and the controller (see summit_xl_control/config/summit_xl_control.yaml)-->
-    <!-- <transmission name="${robot_id}_wheel_joint_trans">
-      <type>transmission_interface/SimpleTransmission</type>
-      <joint name="${robot_id}_wheel_joint" >
-        <hardwareInterface>hardware_interface/VelocityJointInterface</hardwareInterface>
-      </joint>
-      <actuator name="${robot_id}_wheel_joint_motor">
-         <mechanicalReduction>1</mechanicalReduction>
-      </actuator>
-    </transmission> -->
     <gazebo reference="${robot_id}_wheel_link">
       <mu1>0.90</mu1>
@@ -83,5 +63,4 @@
       <kd>8.25e1</kd>
       <fdir1>0 0 0</fdir1>
-      <maxContacts>4</maxContacts>
     </gazebo>
   </xacro:macro>
